File: Jacks/output.kicad_sch (KiCad schematic)
At the start: 16 parts, among them Q301 DMC3071LVT, Q302 DMC3071LVT

Commit message: Trial attempt at different analog rail filtering
This does the +VA net a bit differently: by using a common collector
series follower transistor I can use much bigger resistors in the
lowpass filter because the current through the resistor is just the tiny
base current.

In fact, let's just make it the main filtering stage, and share the
resulting +VA rail for both the input stage and the output bias.  They
both need on the order of one mA of current, so assuming a DC current
gain (whether you call it h_{FE} or Beta) of roughly one hundred, we can
easily use a couple of 2k2 resistors and make it a 2nd order filter.

(The original used a single 220 Ohm resistor, so this increases that by
a factor of twenty, but then the h_{FE} will more than make up for it)

Of course, the small viltage drop over the resistors will now be almost
entirely dwarfed by the V_{BE} voltage drop of the transistor.  But if
it gives us a nice stable analog voltage rail, it should be worth the
small voltage drop.

I use a MOSFET for reverse polarity protection because I don't like the
voltage drop of a simple diode, but that's because the voltage drop
there would be just a negative.  Here there's a _reason_ for a voltage
drop.

Of course, I don't know how much it really helps with noise, but it
looks good in simulation, and I'm willing to at least do a test board
for this.

I'm just using the BC846 BJT I already have around.  It's a very average
cheap general-purpose transistor, I have no idea if this is any good.

Live and learn.  That's still the point of the whole project, after all.

While doing random trials, this also ends up DC-coupling the input side.
I probably shouldn't do two independent changes like this, but I'm too
lazy to do two separate boards.

Talking about separate boards: I wish KiCad had some good way to share
common circuits (some kind of "combination symbol" concept or something)
so that you could do explicitly different boards without having to
either do duplicate board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
Parts:
- removed C306: 10uF, Capacitor_SMD:C_1206_3216Metric, symbol Device:C
- removed R307: 2k2, Resistor_SMD:R_0805_2012Metric, symbol Device:R
- C301, C302, C303: value 4.7uF -> 1uF
- C304: value 150pF -> 220pF
- R304: value 1k -> 2k2
- R306: value 2k2 -> 4k7
- renumbered R308 to R307
Connections:
- net VBIAS: now also C305.2, R306.1
- net VIN renamed +VA
Other:
- moved on the sheet: C305, R306
