File: Jacks/Jacks.kicad_pcb (KiCad board)
At the start: 2 copper layers, 45 x 27.5 mm, 42 parts, among them J101 Barrel_Jack_Switch, J102 AudioJack2_Ground, J103 AudioJack2_Ground, J104 Conn_02x05_Odd_Even, Q101 DMC3071LVT, Q102 BC846, Q201 LS844, Q301 DMC3071LVT, Q302 DMC3071LVT

Commit message: Add ugly 3d model to DC barrel jack
Based on the Würth datasheet:

   https://www.we-online.com/components/products/datasheet/694106301002.pdf

and my stumbling attempts at generating a STEP file with openscad and
freecad.

This time I couldn't get rid of the "hole turns into a plug" problem
with the freecad STEP file exprt, so once again the model looks fine in
both openscad and in freecad, but the STEP export just looks wrong with
no hole for the power plug.

There's some subtle order of operations bug thing going on.  But I'll
use it as a way to distract from the ugliness of the model: everybody
will just look at the lack of hole for the plug, and overlook the harsh
edges.

Also: dazzle them with colors.  That's the trick.  Nobody will question
my mad design skillz when it's colorized and there are obvious freecad
export issues.

Signed-off-by: Linus Torvalds <torvalds@linux-foundation.org>
Parts:
- J101: footprint Connector_BarrelJack:BarrelJack_Wuerth_6941xx301002 -> Mylib:Wurth WR-DC 2.1mm Power Jack
