File: 1590A/Base/sim.kicad_sch (KiCad schematic)
At the start: 13 parts

Commit message: Update 1590A board
I really wanted to use the stomp switch board, but I didn't find any
sane connectors that are convenient and fit.

So I just updated this board to have the stomp switch directly on the
board instead.  I'd love to re-use stomp switches after I have made a
(bad) design and tested it, but the pain just doesn't seem worth it.

That means that I could just have used a traditional latching 3PDT, but
instead this sticks to the electronic switching with a momentary switch.
Because the whole point is the circuit, not sanity.

Add another openscad 3d model for this stomp switch thing.

Signed-off-by: Linus Torvalds <torvalds@linux-foundation.org>
Parts:
- renumbered R1 to R401, V402 to V401, V403 to V402, V404 to V403, V405 to V404, V406 to V405, V407 to V406, V408 to V407
Changed lines of the file:
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@@
 		(on_board no)
 		(dnp no)
-		(property "Reference" "V406"
+		(property "Reference" "V405"
 			(at 130.81 105.2801 0)
 			(effects
@@
 			(project "Buffered"
 				(path "/9e337e0b-885b-4d2b-99a2-62cdd082c615/a1084b87-85fd-4b63-8fe4-8749c999d338"
-					(reference "V406")
+					(reference "V405")
 					(unit 1)
 				)
@@
 		(on_board no)
 		(dnp no)
-		(property "Reference" "V408"
+		(property "Reference" "V407"
 			(at 207.01 48.1301 0)
 			(effects
@@
 			(project "Buffered"
 				(path "/9e337e0b-885b-4d2b-99a2-62cdd082c615/a1084b87-85fd-4b63-8fe4-8749c999d338"
-					(reference "V408")
+					(reference "V407")
 					(unit 1)
 				)
@@
 		(on_board no)
 		(dnp no)
-		(property "Reference" "V403"
+		(property "Reference" "V402"
 			(at 34.29 49.4001 0)
 			(effects
@@
 			(project "Buffered"
 				(path "/9e337e0b-885b-4d2b-99a2-62cdd082c615/a1084b87-85fd-4b63-8fe4-8749c999d338"
-					(reference "V403")
+					(reference "V402")
 					(unit 1)
 				)
@@
 		(on_board no)
 		(dnp yes)
-		(property "Reference" "R1"
+		(property "Reference" "R401"
 			(at 29.21 129.5399 0)
 			(effects
@@
 			(project "Base"
 				(path "/9e337e0b-885b-4d2b-99a2-62cdd082c615/a1084b87-85fd-4b63-8fe4-8749c999d338"
-					(reference "R1")
+					(reference "R401")
 					(unit 1)
 				)
@@
 		(on_board no)
 		(dnp no)
-		(property "Reference" "V407"
+		(property "Reference" "V406"
 			(at 132.08 48.1301 0)
 			(effects
@@
 			(project "Buffered"
 				(path "/9e337e0b-885b-4d2b-99a2-62cdd082c615/a1084b87-85fd-4b63-8fe4-8749c999d338"
-					(reference "V407")
+					(reference "V406")
 					(unit 1)
 				)
@@
 		(dnp no)
 		(fields_autoplaced yes)
-		(property "Reference" "V402"
+		(property "Reference" "V401"
 			(at 34.29 37.9701 0)
 			(effects
@@
 			(project "Buffered"
 				(path "/9e337e0b-885b-4d2b-99a2-62cdd082c615/a1084b87-85fd-4b63-8fe4-8749c999d338"
-					(reference "V402")
+					(reference "V401")
 					(unit 1)
 				)
@@
 		(on_board no)
 		(dnp no)
-		(property "Reference" "V405"
+		(property "Reference" "V404"
 			(at 34.29 73.5301 0)
 			(effects
@@
 			(project "Buffered"
 				(path "/9e337e0b-885b-4d2b-99a2-62cdd082c615/a1084b87-85fd-4b63-8fe4-8749c999d338"
-					(reference "V405")
+					(reference "V404")
 					(unit 1)
 				)
@@
 		(on_board no)
 		(dnp no)
-		(property "Reference" "V404"
+		(property "Reference" "V403"
 			(at 34.29 62.1001 0)
 			(effects
@@
 			(project "Buffered"
 				(path "/9e337e0b-885b-4d2b-99a2-62cdd082c615/a1084b87-85fd-4b63-8fe4-8749c999d338"
-					(reference "V404")
+					(reference "V403")
 					(unit 1)
 				)
