File: 1590A/Base/output.kicad_sch (KiCad schematic)
At the start: 20 parts, among them Q301 DMC3071LVT, Q302 DMC3071LVT, Q303 DMC3071LVT

Commit message: Update 1590A board
I really wanted to use the stomp switch board, but I didn't find any
sane connectors that are convenient and fit.

So I just updated this board to have the stomp switch directly on the
board instead.  I'd love to re-use stomp switches after I have made a
(bad) design and tested it, but the pain just doesn't seem worth it.

That means that I could just have used a traditional latching 3PDT, but
instead this sticks to the electronic switching with a momentary switch.
Because the whole point is the circuit, not sanity.

Add another openscad 3d model for this stomp switch thing.

Signed-off-by: Linus Torvalds <torvalds@linux-foundation.org>
Parts:
- renumbered R312 to R311
Changed lines of the file:
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@@
 		(dnp no)
 		(fields_autoplaced yes)
-		(property "Reference" "R312"
+		(property "Reference" "R311"
 			(at 255.27 85.0899 0)
 			(effects
@@
 			(project "Base"
 				(path "/9e337e0b-885b-4d2b-99a2-62cdd082c615/82119736-3682-4322-9383-b4b2debfc9f1"
-					(reference "R312")
+					(reference "R311")
 					(unit 1)
 				)
