File: 1590B/Base/output.kicad_sch (KiCad schematic)
At the start: 14 parts, among them Q301 DMC3071LVT, Q302 DMC3071LVT

Commit message: Add 1590B base board design
This integrates the stomp switch and the Daisy Seed with the jacks on
the base board, because connecting things up was a bigger pain than just
integrating everything.

The end result mostly matches the 3d model in the Template directory.

As a result of the integration, this also removes the separate Jacks,
Daisy Seed and Stomp boards: they are all parts of the board here.

Signed-off-by: Linus Torvalds <torvalds@linux-foundation.org>
Parts:
- C304: value 220pF -> 1nF
- R304: value 2k2 -> 3k3
Changed lines of the file:
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@@
 	(generator_version "9.0")
 	(paper "A4")
-	(text_box "Output switching\n\nUse series MOSFETs to switch signals on and off. \n\nUse complementary MOSFETS so that we can just use one single gate voltage for both signals.\n\nBig gate resistor to slow down switching and minimize popping\n"
+	(text_box "Output switching\n\nUse series MOSFETs to switch signals on and off. \n\nUse complementary MOSFETS so that we can just use one single gate voltage for both signals.\n\nBig gate resistor to slow down switching and minimize popping\n\n3k3 / 1nF is a 48kHz lowpass filter at output\n"
 		(exclude_from_sim no)
 		(at 14.605 14.605 0)
@@
 			)
 		)
-		(property "Value" "2k2"
+		(property "Value" "3k3"
 			(at 116.84 74.93 90)
 			(effects
@@
 			)
 		)
-		(property "Value" "220pF"
+		(property "Value" "1nF"
 			(at 121.92 87.6299 0)
 			(effects
