File: 1590B/Base/Base.kicad_sch (KiCad schematic)
At the start: 13 parts, among them J101 Barrel_Jack_Switch, J102 AudioJack3_SwitchTR, J103 AudioJack3_SwitchTR, Q101 PMV250, Q102 BC846

Commit message: Update 1590B board for sanity
I had entirely forgotten the activity LED, which was really annoying
when testing.

Also, while the transistor follower / capacitor multiplier on the analog
power supply was interesting for some low frequency power supply ripple
removal in simulation, it doesn't actually make any sense with any
modern power supply, so just do a regular RC filter for high
frequencies, which is what actually matters.

Together with the fixed potentiometer board, I think this should now
work nicely.

Famous last words.

Signed-off-by: Linus Torvalds <torvalds@linux-foundation.org>
Parts:
- removed C101: 10uF, Capacitor_SMD:C_1206_3216Metric, symbol Device:C
- removed Q102: BC846, Package_TO_SOT_SMD:SOT-23, symbol Transistor_BJT:BC846
- removed R106, R107: 2k2, Resistor_SMD:R_0805_2012Metric, symbol Device:R
- added C104: 1uF, Capacitor_SMD:C_1206_3216Metric, symbol Device:C
- added FB101: FerriteBead, Inductor_SMD:L_1206_3216Metric, symbol Device:FerriteBead
- added R102: 100R, Resistor_SMD:R_0805_2012Metric, symbol Device:R
- renumbered Box102 to Box101, C104 to C101
Connections:
- net +VA: now also C104.2, FB101.1; no longer C102.1
- net GND: now also C102.1, C103.1, C104.1; no longer C102.2, C103.2
- net PWRIN: now also C102.2, R102.1
- new net: C103.2, FB101.2, R102.2
