File: RP2354A/tac5112.kicad_sch (KiCad schematic)
At the start: 9 parts, among them U4 TAC5112

Commit message: Rename the "JLCPCB" property as "LCSC PN"
That's apparently the standard way for the 'JLCPCB Fabrication Toolkit'
scripting.  At least for the first time, I want to cross-check with the
scripting, even if I might not necessarily use it as-is.

Signed-off-by: Linus Torvalds <torvalds@linux-foundation.org>
Parts:
- C25, C26, C29: JLCPCB C91606 -> (none); LCSC PN (none) -> C91606
- C27, C28, C30: JLCPCB C1525 -> (none); LCSC PN (none) -> C1525
- C31, C32: JLCPCB C519560 -> (none); LCSC PN (none) -> C519560
- U4: JLCPCB C44853692 -> (none); LCSC PN (none) -> C44853692
Changed lines of the file:
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@@
 			)
 		)
-		(property "JLCPCB" "C1525"
+		(property "LCSC PN" "C1525"
 			(at 93.98 34.29 0)
 			(effects
@@
 			)
 		)
-		(property "JLCPCB" "C519560"
+		(property "LCSC PN" "C519560"
 			(at 180.34 34.29 0)
 			(effects
@@
 			)
 		)
-		(property "JLCPCB" "C91606"
+		(property "LCSC PN" "C91606"
 			(at 137.16 34.29 0)
 			(effects
@@
 			)
 		)
-		(property "JLCPCB" "C1525"
+		(property "LCSC PN" "C1525"
 			(at 78.74 34.29 0)
 			(effects
@@
 			)
 		)
-		(property "JLCPCB" "C519560"
+		(property "LCSC PN" "C519560"
 			(at 163.83 34.29 0)
 			(effects
@@
 			)
 		)
-		(property "JLCPCB" "C91606"
+		(property "LCSC PN" "C91606"
 			(at 46.99 34.29 0)
 			(effects
@@
 			)
 		)
-		(property "JLCPCB" "C91606"
+		(property "LCSC PN" "C91606"
 			(at 63.5 34.29 0)
 			(effects
@@
 			)
 		)
-		(property "JLCPCB" "C1525"
+		(property "LCSC PN" "C1525"
 			(at 144.78 34.29 0)
 			(effects
@@
 			)
 		)
-		(property "JLCPCB" "C44853692"
+		(property "LCSC PN" "C44853692"
 			(at 86.36 93.98 0)
 			(effects
