File: 1590LB/Boost/Boost.kicad_sch (KiCad schematic)
At the start: 22 parts, among them J101 Barrel_Jack_Switch, J102 AudioJack2_SwitchT, J103 AudioJack2_SwitchT, Q101 PMV250, SW101 SW_DPDT_x2

Commit message: Make the boost circuit a bit more interesting
The clean boost with some clipping was very boring, both from a sound
and a circuit standpoint.

This one isn't any better from a sound standpoint, but at least it's a
bit more interesting.  Instead of a boost pot and clipping diodes, this
has a pot that affects the biasing of the input JFET, and a fixed 10x
voltage boost with a final volume pot.

End result: it also clips, but the clipping is based on how badly the
input transistor is biased, so now you have a bit more control over the
result.

Useful? No.  But I'm back to using discrete components, because the
whole op-amp thing was just too boring.  If I want to use pre-made
circuits, I can do that on the MCU board, let's keep the analog boards
discrete.

That said, I've made the resistors and capacitors small, because I'll
just use this one for the JLCPCB assembly testing.  I did send off a
copy of the MCU board too, which is probably completely stupid - the
first PCBA board I do shouldn't have been that complex.  But maybe it
works (after I figure out the programming - even if the board is fine,
I'll have to do the SW side too to even test it).

Anyway, this one I can have assembled - and test - without then having
to write any code for various i2s things that I have no idea about.

Oh, and I still call this a "1590LB" boost board, even though I actually
ended up deciding that I'll just 3D-print the enclosure.  So it's not
really a 1590LB, it's a 45x50mm board that I'll just print a custom
enclosure for.  I actually really liked how one of my test enclosures
ended up looking, and not being limited to standard aluminum boxes is
liberating.

Signed-off-by: Linus Torvalds <torvalds@linux-foundation.org>
Parts:
- removed Box101: 1590LB, Mylib:1590LB, symbol Mylib:Enclosure_1590LB
- removed C105: 10uF, Capacitor_SMD:C_1206_3216Metric, symbol Device:C
- removed C106: 1uF, Capacitor_SMD:C_1206_3216Metric, symbol Device:C
- removed FB101: FerriteBead, Inductor_SMD:L_1206_3216Metric, symbol Device:FerriteBead
- removed R107: 1MEG, Resistor_SMD:R_0805_2012Metric, symbol Device:R
- removed R109: 100R, Resistor_SMD:R_0805_2012Metric, symbol Device:R
- added C4: 10uF, Capacitor_SMD:C_0603_1608Metric, symbol Device:C
- added R5: 33R, Resistor_SMD:R_0402_1005Metric, symbol Device:R
- added R7: 10k, Resistor_SMD:R_0402_1005Metric, symbol Device:R
- added RV1: 100k, Mylib:Potentiometer_9mm_MP, symbol Device:R_Potentiometer_MountingPin
- C1: renamed from C101; footprint Capacitor_SMD:C_1206_3216Metric -> Capacitor_SMD:C_0603_1608Metric
- C2: renamed from C102; footprint Capacitor_SMD:C_0805_2012Metric -> Capacitor_SMD:C_0402_1005Metric
- C3: renamed from C107; footprint Capacitor_SMD:C_1206_3216Metric -> Capacitor_SMD:C_0603_1608Metric
- C5: renamed from C103; value 4.7uF -> 1uF; footprint Capacitor_SMD:C_1206_3216Metric -> Capacitor_SMD:C_0603_1608Metric
- C6: renamed from C104; footprint Capacitor_SMD:C_1206_3216Metric -> Capacitor_SMD:C_0402_1005Metric
- R1: renamed from R111; footprint Resistor_SMD:R_0805_2012Metric -> Resistor_SMD:R_0402_1005Metric
- R2: renamed from R101; footprint Resistor_SMD:R_0805_2012Metric -> Resistor_SMD:R_0402_1005Metric
- R3: renamed from R102; footprint Resistor_SMD:R_0805_2012Metric -> Resistor_SMD:R_0402_1005Metric
- R4: renamed from R103; footprint Resistor_SMD:R_0805_2012Metric -> Resistor_SMD:R_0402_1005Metric
- R6: renamed from R108; footprint Resistor_SMD:R_0805_2012Metric -> Resistor_SMD:R_0402_1005Metric
- renumbered D101 to D1, J101 to J1, J102 to J2, J103 to J3, Q101 to Q1, SW101 to SW1
Connections:
- net +VA: now also C4.2, R5.1
- net GND: now also C4.1, R7.2, RV1.MP (MountPin)
- net OUT^{STOMP}: now also RV1.2; no longer C6.2, R6.2
- net VIN: now also R5.2
- new net: C6.2, R6.2, RV1.3
- new net: R7.1, RV1.1
Other:
- note added: "Silly dirt pedal. The clean op-amp version was just too boring for words. This one just does a 10x signal amplification, with bias control to change the clipping"
- note removed: "Boost pedal with discrete op-amp'ish circuit"
- moved on the sheet: C3, C6, J2, J3, Q1, R4, R6, SW1B

Commit message: 1590LB boost / dirt circuit: add LCSC parts numbers
The PMV250 PNP high-side MOSFET is now a AO3401A, and the BC847C is now
a BC849C instead.  Because those were what I went with at JLCPCB.

It's kind of stupid to have this assembled by machine, since it would be
easy to do by hand (admittedly with slightly different size choices),
and this is not a particularly good design for JLCPCB anyway since all
those matched dual transistors are extended parts etc.

But the point was mainly to do PCBA with a simple board so that I can
actually verify that I did it right.  When the RP2354A comes back, it
will take some coding to get it to do anything at all, so if I screwed
up the hw, it's not going to be as obvious (unless I did it really badly
and the magic smoke escapes).

With this, it's going to be pretty obvious when it doesn't work that my
hw design is just wrong.  Or maybe it works fine - it _should_.  I've
successfully tested a very similar basic circuit, but this does have a
different JFET and some other changes.

Anyway, it's sent off.  When I get back home from travels, I should have
something to test.

Signed-off-by: Linus Torvalds <torvalds@linux-foundation.org>
Parts:
- C1, C5: LCSC PN (none) -> C519560
- C2: LCSC PN (none) -> C710836
- C3, C4: LCSC PN (none) -> C91606
- C6: LCSC PN (none) -> C1523
- Q1: LCSC PN (none) -> C15127
- R1, R6: LCSC PN (none) -> C25890
- R2: LCSC PN (none) -> C26083
- R3: LCSC PN (none) -> C11702
- R4: LCSC PN (none) -> C25741
- R5: LCSC PN (none) -> C25105
- R7: LCSC PN (none) -> C25744
Changed lines of the file:
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@@
 			)
 		)
+		(property "LCSC PN" "C519560"
+			(at 53.34 96.52 90)
+			(effects
+				(font
+					(size 1.27 1.27)
+				)
+				(hide yes)
+			)
+		)
 		(pin "2"
 		)
@@
 			)
 		)
+		(property "LCSC PN" "C25890"
+			(at 29.21 158.75 90)
+			(effects
+				(font
+					(size 1.27 1.27)
+				)
+				(hide yes)
+			)
+		)
 		(pin "2"
 		)
@@
 			)
 		)
+		(property "LCSC PN" "C1523"
+			(at 176.53 102.87 0)
+			(effects
+				(font
+					(size 1.27 1.27)
+				)
+				(hide yes)
+			)
+		)
 		(pin "2"
 		)
@@
 			)
 		)
+		(property "LCSC PN" "C11702"
+			(at 64.77 96.52 90)
+			(effects
+				(font
+					(size 1.27 1.27)
+				)
+				(hide yes)
+			)
+		)
 		(pin "1"
 		)
@@
 			)
 		)
+		(property "LCSC PN" "C710836"
+			(at 73.66 104.14 0)
+			(effects
+				(font
+					(size 1.27 1.27)
+				)
+				(hide yes)
+			)
+		)
 		(pin "2"
 		)
@@
 			)
 		)
+		(property "LCSC PN" ""
+			(at 29.21 34.29 0)
+			(effects
+				(font
+					(size 1.27 1.27)
+				)
+				(hide yes)
+			)
+		)
 		(pin "1"
 		)
@@
 			)
 		)
+		(property "LCSC PN" "C91606"
+			(at 88.9 44.45 0)
+			(effects
+				(font
+					(size 1.27 1.27)
+				)
+				(hide yes)
+			)
+		)
 		(pin "2"
 		)
@@
 			)
 		)
+		(property "LCSC PN" "C25744"
+			(at 196.85 111.76 0)
+			(effects
+				(font
+					(size 1.27 1.27)
+				)
+				(hide yes)
+			)
+		)
 		(pin "1"
 		)
@@
 			)
 		)
+		(property "LCSC PN" "C25890"
+			(at 165.1 93.98 90)
+			(effects
+				(font
+					(size 1.27 1.27)
+				)
+				(hide yes)
+			)
+		)
 		(pin "1"
 		)
@@
 			)
 		)
+		(property "LCSC PN" ""
+			(at 49.53 156.21 0)
+			(effects
+				(font
+					(size 1.27 1.27)
+				)
+				(hide yes)
+			)
+		)
 		(pin "2"
 		)
@@
 			)
 		)
+		(property "LCSC PN" ""
+			(at 168.91 45.72 0)
+			(effects
+				(font
+					(size 1.27 1.27)
+				)
+				(hide yes)
+			)
+		)
 		(pin "T"
 		)
@@
 			)
 		)
+		(property "LCSC PN" ""
+			(at 196.85 102.87 0)
+			(effects
+				(font
+					(size 1.27 1.27)
+				)
+				(hide yes)
+			)
+		)
 		(pin "2"
 		)
@@
 			)
 		)
+		(property "LCSC PN" "C25741"
+			(at 72.39 46.99 0)
+			(effects
+				(font
+					(size 1.27 1.27)
+				)
+				(hide yes)
+			)
+		)
 		(pin "2"
 		)
@@
 			)
 		)
+		(property "LCSC PN" "C91606"
+			(at 116.84 48.26 0)
+			(effects
+				(font
+					(size 1.27 1.27)
+				)
+				(hide yes)
+			)
+		)
 		(pin "2"
 		)
@@
 			)
 		)
+		(property "LCSC PN" ""
+			(at 39.37 156.21 0)
+			(effects
+				(font
+					(size 1.27 1.27)
+				)
+				(hide yes)
+			)
+		)
 		(pin "3"
 		)
@@
 			)
 		)
+		(property "LCSC PN" ""
+			(at 198.12 45.72 0)
+			(effects
+				(font
+					(size 1.27 1.27)
+				)
+				(hide yes)
+			)
+		)
 		(pin "T"
 		)
@@
 			)
 		)
+		(property "LCSC PN" "C25105"
+			(at 116.84 38.1 0)
+			(effects
+				(font
+					(size 1.27 1.27)
+				)
+				(hide yes)
+			)
+		)
 		(pin "1"
 		)
@@
 			)
 		)
+		(property "LCSC PN" "C519560"
+			(at 153.67 93.98 90)
+			(effects
+				(font
+					(size 1.27 1.27)
+				)
+				(hide yes)
+			)
+		)
 		(pin "2"
 		)
@@
 			)
 		)
+		(property "LCSC PN" ""
+			(at 83.82 156.21 0)
+			(effects
+				(font
+					(size 1.27 1.27)
+				)
+				(hide yes)
+			)
+		)
 		(pin "3"
 		)
@@
 			)
 		)
+		(property "LCSC PN" "C15127"
+			(at 72.39 35.56 0)
+			(effects
+				(font
+					(size 1.27 1.27)
+				)
+				(hide yes)
+			)
+		)
 		(pin "2"
 		)
@@
 			(at 45.72 104.14 0)
 			(effects
+				(font
+					(size 1.27 1.27)
+				)
+				(hide yes)
+			)
+		)
+		(property "LCSC PN" "C26083"
+			(at 45.72 104.14 0)
+			(effects
