File: 1590LB/Boost/sim.kicad_sch (KiCad schematic)
At the start: 12 parts

Commit message: Make the boost circuit a bit more interesting
The clean boost with some clipping was very boring, both from a sound
and a circuit standpoint.

This one isn't any better from a sound standpoint, but at least it's a
bit more interesting.  Instead of a boost pot and clipping diodes, this
has a pot that affects the biasing of the input JFET, and a fixed 10x
voltage boost with a final volume pot.

End result: it also clips, but the clipping is based on how badly the
input transistor is biased, so now you have a bit more control over the
result.

Useful? No.  But I'm back to using discrete components, because the
whole op-amp thing was just too boring.  If I want to use pre-made
circuits, I can do that on the MCU board, let's keep the analog boards
discrete.

That said, I've made the resistors and capacitors small, because I'll
just use this one for the JLCPCB assembly testing.  I did send off a
copy of the MCU board too, which is probably completely stupid - the
first PCBA board I do shouldn't have been that complex.  But maybe it
works (after I figure out the programming - even if the board is fine,
I'll have to do the SW side too to even test it).

Anyway, this one I can have assembled - and test - without then having
to write any code for various i2s things that I have no idea about.

Oh, and I still call this a "1590LB" boost board, even though I actually
ended up deciding that I'll just 3D-print the enclosure.  So it's not
really a 1590LB, it's a 45x50mm board that I'll just print a custom
enclosure for.  I actually really liked how one of my test enclosures
ended up looking, and not being limited to standard aluminum boxes is
liberating.

Signed-off-by: Linus Torvalds <torvalds@linux-foundation.org>
Parts:
- removed R301: 1k, symbol Device:R
- renumbered R302 to R14, R303 to R15, R304 to R16, R305 to R17, V301 to V1, V302 to V2, V303 to V3, V304 to V4, V305 to V5, V306 to V6, V307 to V7
Changed lines of the file:
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@@
 		(title "Simulation infrastructure")
 	)
-	(text_box "Simulate effect power use: 9V over 150 Ohm is 60mA.\nPower rail has 60Hz ripple, 2.5kHz DC converter noise\n\nLED simulated on for random current check"
+	(text_box "Simulate effect power use: 9V over 150 Ohm is 60mA.\nPower rail has 60Hz ripple, 2.5kHz DC converter noise"
 		(exclude_from_sim no)
 		(at 13.97 14.605 0)
@@
 		)
 	)
-	(global_label "VIN"
-		(shape input)
-		(at 68.58 43.18 90)
-		(fields_autoplaced yes)
-		(effects
-			(font
-				(size 1.27 1.27)
-			)
-			(justify left)
-		)
-		(property "Intersheetrefs" "${INTERSHEET_REFS}"
-			(at 68.58 37.1709 90)
-			(effects
-				(font
-					(size 1.27 1.27)
-				)
-				(justify left)
-				(hide yes)
-			)
-		)
-	)
 	(global_label "IN^{EFF}"
 		(shape input)
@@
 		(dnp no)
 		(fields_autoplaced yes)
-		(property "Reference" "#PWR0405"
+		(property "Reference" "#PWR025"
 			(at 127 119.38 0)
 			(effects
@@
 			(project "Stomp"
 				(path "/9e337e0b-885b-4d2b-99a2-62cdd082c615/a1084b87-85fd-4b63-8fe4-8749c999d338"
-					(reference "#PWR0405")
-					(unit 1)
-				)
-			)
-		)
-	)
-	(symbol
-		(lib_id "power:GND")
-		(at 68.58 50.8 0)
-		(unit 1)
-		(exclude_from_sim no)
-		(in_bom yes)
-		(on_board yes)
-		(dnp no)
-		(fields_autoplaced yes)
-		(property "Reference" "#PWR0403"
-			(at 68.58 57.15 0)
-			(effects
-				(font
-					(size 1.27 1.27)
-				)
-				(hide yes)
-			)
-		)
-		(property "Value" "GND"
-			(at 68.58 55.88 0)
-			(effects
-				(font
-					(size 1.27 1.27)
-				)
-			)
-		)
-		(property "Footprint" ""
-			(at 68.58 50.8 0)
-			(effects
-				(font
-					(size 1.27 1.27)
-				)
-				(hide yes)
-			)
-		)
-		(property "Datasheet" ""
-			(at 68.58 50.8 0)
-			(effects
-				(font
-					(size 1.27 1.27)
-				)
-				(hide yes)
-			)
-		)
-		(property "Description" "Power symbol creates a global label with name \"GND\" , ground"
-			(at 68.58 50.8 0)
-			(effects
-				(font
-					(size 1.27 1.27)
-				)
-				(hide yes)
-			)
-		)
-		(pin "1"
-		)
-		(instances
-			(project "Stomp"
-				(path "/9e337e0b-885b-4d2b-99a2-62cdd082c615/a1084b87-85fd-4b63-8fe4-8749c999d338"
-					(reference "#PWR0403")
+					(reference "#PWR025")
 					(unit 1)
 				)
@@
 		(on_board no)
 		(dnp no)
-		(property "Reference" "V305"
+		(property "Reference" "V5"
 			(at 130.81 105.2801 0)
 			(effects
@@
 			(project "Stomp"
 				(path "/9e337e0b-885b-4d2b-99a2-62cdd082c615/a1084b87-85fd-4b63-8fe4-8749c999d338"
-					(reference "V305")
+					(reference "V5")
 					(unit 1)
 				)
@@
 		(on_board no)
 		(dnp no)
-		(property "Reference" "V307"
+		(property "Reference" "V7"
 			(at 207.01 48.1301 0)
 			(effects
@@
 			(project "Stomp"
 				(path "/9e337e0b-885b-4d2b-99a2-62cdd082c615/a1084b87-85fd-4b63-8fe4-8749c999d338"
-					(reference "V307")
+					(reference "V7")
 					(unit 1)
 				)
@@
 		(dnp yes)
 		(fields_autoplaced yes)
-		(property "Reference" "R303"
+		(property "Reference" "R15"
 			(at 125.73 154.94 90)
 			(effects
@@
 			(project "Stomp"
 				(path "/9e337e0b-885b-4d2b-99a2-62cdd082c615/a1084b87-85fd-4b63-8fe4-8749c999d338"
-					(reference "R303")
+					(reference "R15")
 					(unit 1)
 				)
@@
 		(on_board no)
 		(dnp no)
-		(property "Reference" "V302"
+		(property "Reference" "V2"
 			(at 34.29 57.0201 0)
 			(effects
@@
 			(project "Stomp"
 				(path "/9e337e0b-885b-4d2b-99a2-62cdd082c615/a1084b87-85fd-4b63-8fe4-8749c999d338"
-					(reference "V302")
+					(reference "V2")
 					(unit 1)
 				)
@@
 		(dnp no)
 		(fields_autoplaced yes)
-		(property "Reference" "#PWR0409"
+		(property "Reference" "#PWR028"
 			(at 138.43 161.29 0)
 			(effects
@@
 			(project "Stomp"
 				(path "/9e337e0b-885b-4d2b-99a2-62cdd082c615/a1084b87-85fd-4b63-8fe4-8749c999d338"
-					(reference "#PWR0409")
+					(reference "#PWR028")
 					(unit 1)
 				)
@@
 		(dnp no)
 		(fields_autoplaced yes)
-		(property "Reference" "#PWR0402"
+		(property "Reference" "#PWR024"
 			(at 30.48 97.79 0)
 			(effects
@@
 			(project "Stomp"
 				(path "/9e337e0b-885b-4d2b-99a2-62cdd082c615/a1084b87-85fd-4b63-8fe4-8749c999d338"
-					(reference "#PWR0402")
+					(reference "#PWR024")
 					(unit 1)
 				)
@@
 		(on_board no)
 		(dnp yes)
-		(property "Reference" "R304"
+		(property "Reference" "R16"
 			(at 123.19 167.6399 90)
 			(effects
@@
 			(project "Stomp"
 				(path "/9e337e0b-885b-4d2b-99a2-62cdd082c615/a1084b87-85fd-4b63-8fe4-8749c999d338"
-					(reference "R304")
+					(reference "R16")
 					(unit 1)
 				)
@@
 		(dnp no)
 		(fields_autoplaced yes)
-		(property "Reference" "#PWR0404"
+		(property "Reference" "#PWR027"
 			(at 138.43 149.86 0)
 			(effects
@@
 			(project "Stomp"
 				(path "/9e337e0b-885b-4d2b-99a2-62cdd082c615/a1084b87-85fd-4b63-8fe4-8749c999d338"
-					(reference "#PWR0404")
+					(reference "#PWR027")
 					(unit 1)
 				)
@@
 		(on_board no)
 		(dnp no)
-		(property "Reference" "V306"
+		(property "Reference" "V6"
 			(at 132.08 48.1301 0)
 			(effects
@@
 			)
 		)
-		(property "Sim.Params" "y1=-0.2 y2=0.2 td=5m tr=25m tf=25m tw=1u per=50m ac=1"
+		(property "Sim.Params" "y1=-0.3 y2=0.3 td=5m tr=25m tf=25m tw=1u per=50m ac=1"
 			(at 104.14 67.564 0)
 			(effects
@@
 			(project "Stomp"
 				(path "/9e337e0b-885b-4d2b-99a2-62cdd082c615/a1084b87-85fd-4b63-8fe4-8749c999d338"
-					(reference "V306")
+					(reference "V6")
 					(unit 1)
 				)
@@
 		(dnp no)
 		(fields_autoplaced yes)
-		(property "Reference" "#PWR0406"
+		(property "Reference" "#PWR026"
 			(at 128.27 62.23 0)
 			(effects
@@
 			(project "Stomp"
 				(path "/9e337e0b-885b-4d2b-99a2-62cdd082c615/a1084b87-85fd-4b63-8fe4-8749c999d338"
-					(reference "#PWR0406")
+					(reference "#PWR026")
 					(unit 1)
 				)
@@
 		(dnp no)
 		(fields_autoplaced yes)
-		(property "Reference" "V301"
+		(property "Reference" "V1"
 			(at 34.29 45.5901 0)
 			(effects
@@
 			(project "Stomp"
 				(path "/9e337e0b-885b-4d2b-99a2-62cdd082c615/a1084b87-85fd-4b63-8fe4-8749c999d338"
-					(reference "V301")
+					(reference "V1")
 					(unit 1)
 				)
@@
 		(on_board no)
 		(dnp no)
-		(property "Reference" "V304"
+		(property "Reference" "V4"
 			(at 34.29 81.1501 0)
 			(effects
@@
 			(project "Stomp"
 				(path "/9e337e0b-885b-4d2b-99a2-62cdd082c615/a1084b87-85fd-4b63-8fe4-8749c999d338"
-					(reference "V304")
+					(reference "V4")
 					(unit 1)
 				)
@@
 		(on_board no)
 		(dnp no)
-		(property "Reference" "V303"
+		(property "Reference" "V3"
 			(at 34.29 69.7201 0)
 			(effects
@@
 			(project "Stomp"
 				(path "/9e337e0b-885b-4d2b-99a2-62cdd082c615/a1084b87-85fd-4b63-8fe4-8749c999d338"
-					(reference "V303")
-					(unit 1)
-				)
-			)
-		)
-	)
-	(symbol
-		(lib_id "Device:R")
-		(at 68.58 46.99 180)
-		(unit 1)
-		(exclude_from_sim no)
-		(in_bom no)
-		(on_board no)
-		(dnp yes)
-		(fields_autoplaced yes)
-		(property "Reference" "R301"
-			(at 71.12 45.7199 0)
-			(effects
-				(font
-					(size 1.27 1.27)
-				)
-				(justify right)
-			)
-		)
-		(property "Value" "1k"
-			(at 71.12 48.2599 0)
-			(effects
-				(font
-					(size 1.27 1.27)
-				)
-				(justify right)
-			)
-		)
-		(property "Footprint" ""
-			(at 70.358 46.99 90)
-			(effects
-				(font
-					(size 1.27 1.27)
-				)
-				(hide yes)
-			)
-		)
-		(property "Datasheet" "~"
-			(at 68.58 46.99 0)
-			(effects
-				(font
-					(size 1.27 1.27)
-				)
-				(hide yes)
-			)
-		)
-		(property "Description" "Resistor"
-			(at 68.58 46.99 0)
-			(effects
-				(font
-					(size 1.27 1.27)
-				)
-				(hide yes)
-			)
-		)
-		(pin "1"
-		)
-		(pin "2"
-		)
-		(instances
-			(project "Stomp"
-				(path "/9e337e0b-885b-4d2b-99a2-62cdd082c615/a1084b87-85fd-4b63-8fe4-8749c999d338"
-					(reference "R301")
+					(reference "V3")
 					(unit 1)
 				)
@@
 		(dnp yes)
 		(fields_autoplaced yes)
-		(property "Reference" "R302"
+		(property "Reference" "R14"
 			(at 125.73 143.51 90)
 			(effects
@@
 			(project "Stomp"
 				(path "/9e337e0b-885b-4d2b-99a2-62cdd082c615/a1084b87-85fd-4b63-8fe4-8749c999d338"
-					(reference "R302")
+					(reference "R14")
 					(unit 1)
 				)
@@
 		(dnp no)
 		(fields_autoplaced yes)
-		(property "Reference" "#PWR0407"
+		(property "Reference" "#PWR029"
 			(at 203.2 62.23 0)
 			(effects
@@
 			(project "Stomp"
 				(path "/9e337e0b-885b-4d2b-99a2-62cdd082c615/a1084b87-85fd-4b63-8fe4-8749c999d338"
-					(reference "#PWR0407")
+					(reference "#PWR029")
 					(unit 1)
 				)
@@
 		(dnp yes)
 		(fields_autoplaced yes)
-		(property "Reference" "R305"
+		(property "Reference" "R17"
 			(at 125.73 180.34 90)
 			(effects
@@
 			(project "Boost"
 				(path "/9e337e0b-885b-4d2b-99a2-62cdd082c615/a1084b87-85fd-4b63-8fe4-8749c999d338"
-					(reference "R305")
+					(reference "R17")
 					(unit 1)
 				)
