File: Hardware/pedal-board/pedal-board.kicad_sch (KiCad schematic)
At the start: 21 parts, among them J1 Conn_01x12_MountingPin, J2 TYPE-C16PIN, J3 BM28B0.6-24DS/2, J4 I2C1, J5 Conn_01x03_Pin, SW1 RotaryEncoder_Switch_MP, SW2 RotaryEncoder_Switch_MP, U1 TLV76733DRVx, U2 USBLC6-2P6

Commit message: Add 47uF hybrid aluminum caps to 3.3V and 5V supplies
This was something I did for the usb-stomp switch with the MIDI
connectors and no UI as a "just because" thing.  I had used that cap on
the board for the audio jacks, so it was on my radar, and I was "let's
do it on the USB board too in case it helps with USB power supply noise".

I just compared the older pedal with the new smaller one, and they are
both very quiet, but the pedal with the UI clearly has some noise when
rotating the effect knob and moving between effects.

It could be just the result of doing the "effect->seq++" when a pot
changes, and the resulting work on the audio core, but I had some
similar noise issues long ago when doing screen updates.  Those seemed
to go away when I switched over to the background i2c DMA updates for
the screen updates, but I wonder if it's the screen itself that just
uses more power when updating.

Because it's not noise from USB power: this happens with the a plain and
fairly quiet 9V guitar pedal power supply.

I don't have a power meter for the 9V side, but when powering the pedals
over USB, the small MIDI version without a display draws around 55mA
according to my USB power meter thing, while the UI version draws
between 72..80mA.

Perhaps even more relevant is that the power draw seems to be related to
how many pixels are lit on the screen: so just switching the display to
an effect with less text on it - without changing which effects are
enabled or not - will consistently make it be around that lower power
draw, while a more active screen will consistently be in the upper
range.

So it doesn't sound entirely crazy to think that it might be some power
supply noise - even if this all should be on the digital 3.3V side, not
the separate analog 3.3V rail on the audio jack board.  Those things
*should* be very well isolated from each other, but there's obviously
the digital i2c and i2s lines that cross that boundary.

Of course, it might be some cross-talk issue with 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
Parts:
- added C5 (x2): 47uF, Capacitor_SMD:CP_Elec_6.3x5.9, symbol Device:C_Polarized
Connections:
- net +3V3: now also C5.1
- net GND: now also C5.2, C5.2
- net VBUS: now also C5.1
