File: Hardware/pedal-board/pedal-board.kicad_sch (KiCad schematic)
At the start: 23 parts, among them J1 Conn_01x12_MountingPin, J2 TYPE-C16PIN, J3 BM28B0.6-24DS/2, J4 I2C1, J5 Conn_01x03_Pin, SW1 RotaryEncoder_Switch_MP, SW2 RotaryEncoder_Switch_MP, U1 TLV76733DRVx, U2 USBLC6-2P6

Commit message: Delete the empty and duplicate schematic fields
Importing parts from SnapEDA and from JLCPCB's library left a pile of
fields behind, and almost none of them ever held anything.  Counting
fields that are *present* makes this look like a naming problem - four
spellings of a manufacturer part number, three of the JLCPCB number -
but counting the ones that are *populated* says something simpler:

  LCSC PN     351 present   349 filled
  LCSC        141 present     1 filled
  LSCS PN      55 present     0 filled
  MP          113 present     0 filled
  MF          113 present     0 filled
  VENDOR      113 present     0 filled
  Field6      126 present     0 filled

So LCSC PN was already the one that mattered, and the rest is debris.
This removes 1964 property blocks: fourteen field names that are empty
on every symbol in every project, plus LCSC and LSCS PN, plus JLCPCB -
which was populated on fifteen symbols and agreed with LCSC PN on all
fifteen.  The one populated LCSC carried the same value as its own
LCSC PN, so nothing is lost.

None of it comes from the symbol libraries: only Reference, Value,
Footprint, Datasheet and Description are defined there, so these do not
grow back when a symbol is updated from its library.  One exception
worth knowing about - a single library symbol does define JLCPCB, so
that one can return, and cleaning it means editing the .kicad_sym.

Prec on the rotary board's R104 goes too; it said "1%", which is now in
that part's entry in Hardware/parts.txt.

Verified by exporting a netlist for each of the seven projects before
and after: every net, and every pin on every net, is identical.

Signed-off-by: Linus Torvalds <torvalds@linux-foundation.org>
Parts:
- J4: JLCPCB C160404 -> (none)

Commit message: Fill in the manufacturer part numbers from the parts list
Every symbol that carries an LCSC PN now carries the manufacturer's own
part number beside it: 349 of them, against 17 before.  100 went into a
MANUFACTURER_PART_NUMBER field that already existed and was empty, and
232 needed the field creating, hidden, next to the LCSC PN it came
from.  Fifteen already agreed and were left alone.

The values come from Hardware/parts.txt, keyed on LCSC PN, taking the
part number as the last whitespace-separated token of each entry's
manufacturer line - which is what that line's shape means.

Two capacitors said "Samsung CL32B226KAJNNNE", with the maker's name
inside the part-number field; they now say CL32B226KAJNNNE like
everything else.  The manufacturer is not duplicated into the
schematics at all - parts.txt holds it, and the part number identifies
the part on its own.

Four one-off field names go with this, their contents now recorded
properly:

  Manufacturer / Part#  on the rotary board's L101, which is the Murata
                        LQM2MPN1R0MGHL
  Manufacutrer          the typo, on two inductors: DFE201612E-2R2M=P2
  Part                  on five Schottkys, saying "LRC LMBR130T1G"

That last one is worth a second look rather than a straight delete.
JLCPCB ships C191023 as a Guangdong Hottech 1N5819WS, so the schematic
was naming a different manufacturer's equivalent from the one actually
fitted.  The part number recorded here is what gets assembled; the
disagreement is written down in parts.txt next to the entry.

Netlists exported for all seven projects before and after: every net
and every pin on every net unchanged.

Signed-off-by: Linus Torvalds <torvalds@linux-foundation.org>
Parts:
- C1, C2, C3, C4: MANUFACTURER_PART_NUMBER (none) -> GRM21BR71E225KE11L
- C5: MANUFACTURER_PART_NUMBER (none) -> EEHZA1V470P
- D1: MANUFACTURER_PART_NUMBER (none) -> LTST-C281KGKT
- J1: MANUFACTURER_PART_NUMBER (none) -> AFH05-S12FIA-1H
- J2: MANUFACTURER_PART_NUMBER (none) -> GT-USB-7051A
- J3: MANUFACTURER_PART_NUMBER (none) -> BM28B0.6-24DS/2-0.35V(51)
- J4: MANUFACTURER_PART_NUMBER (none) -> SM04B-SRSS-TB(LF)(SN)
- R1, R2: MANUFACTURER_PART_NUMBER (none) -> 0402WGF5101TCE
- R3, R4, R5: MANUFACTURER_PART_NUMBER (none) -> 0402WGF1001TCE
- U1: MANUFACTURER_PART_NUMBER (none) -> TLV76733DRVR
- U2: MANUFACTURER_PART_NUMBER (none) -> USBLC6-2P6
Changed lines of the file:
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@@
 			)
 		)
+		(property "MANUFACTURER_PART_NUMBER" "GRM21BR71E225KE11L"
+			(at 228.6 40.64 0)
+			(hide yes)
+			(show_name no)
+			(do_not_autoplace no)
+			(effects
+				(font
+					(size 1.27 1.27)
+				)
+			)
+		)
 		(property "Sim.Library" ""
 			(at 228.6 40.64 0)
@@
 			)
 		)
+		(property "MANUFACTURER_PART_NUMBER" "SM04B-SRSS-TB(LF)(SN)"
+			(at 33.02 142.24 0)
+			(hide yes)
+			(show_name no)
+			(do_not_autoplace no)
+			(effects
+				(font
+					(size 1.27 1.27)
+				)
+			)
+		)
 		(property "Sim.Library" ""
 			(at 33.02 142.24 0)
@@
 			)
 		)
+		(property "MANUFACTURER_PART_NUMBER" "EEHZA1V470P"
+			(at 250.19 82.55 0)
+			(hide yes)
+			(show_name no)
+			(do_not_autoplace no)
+			(effects
+				(font
+					(size 1.27 1.27)
+				)
+			)
+		)
 		(pin "2"
 		)
@@
 			)
 		)
+		(property "MANUFACTURER_PART_NUMBER" "GRM21BR71E225KE11L"
+			(at 254 40.64 0)
+			(hide yes)
+			(show_name no)
+			(do_not_autoplace no)
+			(effects
+				(font
+					(size 1.27 1.27)
+				)
+			)
+		)
 		(property "Sim.Library" ""
 			(at 254 40.64 0)
@@
 			)
 		)
+		(property "MANUFACTURER_PART_NUMBER" "GT-USB-7051A"
+			(at 30.48 40.64 0)
+			(hide yes)
+			(show_name no)
+			(do_not_autoplace no)
+			(effects
+				(font
+					(size 1.27 1.27)
+				)
+			)
+		)
 		(property "Sim.Library" ""
 			(at 30.48 40.64 0)
@@
 			)
 		)
+		(property "MANUFACTURER_PART_NUMBER" "GRM21BR71E225KE11L"
+			(at 25.4 143.51 0)
+			(hide yes)
+			(show_name no)
+			(do_not_autoplace no)
+			(effects
+				(font
+					(size 1.27 1.27)
+				)
+			)
+		)
 		(property "Sim.Library" ""
 			(at 25.4 143.51 0)
@@
 			)
 		)
-		(property "MANUFACTURER_PART_NUMBER" ""
+		(property "MANUFACTURER_PART_NUMBER" "0402WGF1001TCE"
 			(at 142.24 172.72 0)
 			(effects
@@
 			)
 		)
+		(property "MANUFACTURER_PART_NUMBER" "LTST-C281KGKT"
+			(at 189.23 92.71 90)
+			(hide yes)
+			(show_name no)
+			(do_not_autoplace no)
+			(effects
+				(font
+					(size 1.27 1.27)
+				)
+			)
+		)
 		(property "Sim.Library" ""
 			(at 189.23 92.71 90)
@@
 			)
 		)
+		(property "MANUFACTURER_PART_NUMBER" "0402WGF5101TCE"
+			(at 62.23 33.02 90)
+			(hide yes)
+			(show_name no)
+			(do_not_autoplace no)
+			(effects
+				(font
+					(size 1.27 1.27)
+				)
+			)
+		)
 		(pin "1"
 		)
@@
 			)
 		)
+		(property "MANUFACTURER_PART_NUMBER" "USBLC6-2P6"
+			(at 67.31 54.61 0)
+			(hide yes)
+			(show_name no)
+			(do_not_autoplace no)
+			(effects
+				(font
+					(size 1.27 1.27)
+				)
+			)
+		)
 		(pin "4"
 		)
@@
 			)
 		)
+		(property "MANUFACTURER_PART_NUMBER" "TLV76733DRVR"
+			(at 241.3 38.1 0)
+			(hide yes)
+			(show_name no)
+			(do_not_autoplace no)
+			(effects
+				(font
+					(size 1.27 1.27)
+				)
+			)
+		)
 		(property "Sim.Library" ""
 			(at 241.3 38.1 0)
@@
 			)
 		)
+		(property "MANUFACTURER_PART_NUMBER" "0402WGF5101TCE"
+			(at 62.23 30.48 90)
+			(hide yes)
+			(show_name no)
+			(do_not_autoplace no)
+			(effects
+				(font
+					(size 1.27 1.27)
+				)
+			)
+		)
 		(pin "1"
 		)
@@
 			)
 		)
+		(property "MANUFACTURER_PART_NUMBER" "AFH05-S12FIA-1H"
+			(at 165.1 39.37 0)
+			(hide yes)
+			(show_name no)
+			(do_not_autoplace no)
+			(effects
+				(font
+					(size 1.27 1.27)
+				)
+			)
+		)
 		(property "Sim.Library" ""
 			(at 165.1 39.37 0)
@@
 			)
 		)
+		(property "MANUFACTURER_PART_NUMBER" "BM28B0.6-24DS/2-0.35V(51)"
+			(at 110.49 41.91 0)
+			(hide yes)
+			(show_name no)
+			(do_not_autoplace no)
+			(effects
+				(font
+					(size 1.27 1.27)
+				)
+			)
+		)
 		(property "Sim.Library" ""
 			(at 110.49 41.91 0)
@@
 			)
 		)
+		(property "MANUFACTURER_PART_NUMBER" "EEHZA1V470P"
+			(at 231.14 82.55 0)
+			(hide yes)
+			(show_name no)
+			(do_not_autoplace no)
+			(effects
+				(font
+					(size 1.27 1.27)
+				)
+			)
+		)
 		(pin "2"
 		)
@@
 			)
 		)
+		(property "MANUFACTURER_PART_NUMBER" "GRM21BR71E225KE11L"
+			(at 82.55 25.4 0)
+			(hide yes)
+			(show_name no)
+			(do_not_autoplace no)
+			(effects
+				(font
+					(size 1.27 1.27)
+				)
+			)
+		)
 		(property "Sim.Library" ""
 			(at 82.55 25.4 0)
@@
 			)
 		)
-		(property "MANUFACTURER_PART_NUMBER" ""
+		(property "MANUFACTURER_PART_NUMBER" "0402WGF1001TCE"
 			(at 181.61 92.71 0)
 			(effects
@@
 			)
 		)
-		(property "MANUFACTURER_PART_NUMBER" ""
+		(property "MANUFACTURER_PART_NUMBER" "0402WGF1001TCE"
 			(at 111.76 172.72 0)
 			(effects
