File: Hardware/audio-jacks/audio-jacks.kicad_sch (KiCad schematic)
At the start: 59 parts, among them J1 Barrel_Jack_Switch, J2 AudioJack3_SwitchTR, J3 AudioJack3_SwitchTR, J4 Conn_01x12_MountingPin, U1 TLV76750DRVx, U2 OPA2365AIDR, U3 TLV76733DRVx, U4 TAC5242, U5 M24C64-FMH6TG

Commit message: Delete the empty and duplicate schematic fields
Importing parts from SnapEDA and from JLCPCB's library left a pile of
fields behind, and almost none of them ever held anything.  Counting
fields that are *present* makes this look like a naming problem - four
spellings of a manufacturer part number, three of the JLCPCB number -
but counting the ones that are *populated* says something simpler:

  LCSC PN     351 present   349 filled
  LCSC        141 present     1 filled
  LSCS PN      55 present     0 filled
  MP          113 present     0 filled
  MF          113 present     0 filled
  VENDOR      113 present     0 filled
  Field6      126 present     0 filled

So LCSC PN was already the one that mattered, and the rest is debris.
This removes 1964 property blocks: fourteen field names that are empty
on every symbol in every project, plus LCSC and LSCS PN, plus JLCPCB -
which was populated on fifteen symbols and agreed with LCSC PN on all
fifteen.  The one populated LCSC carried the same value as its own
LCSC PN, so nothing is lost.

None of it comes from the symbol libraries: only Reference, Value,
Footprint, Datasheet and Description are defined there, so these do not
grow back when a symbol is updated from its library.  One exception
worth knowing about - a single library symbol does define JLCPCB, so
that one can return, and cleaning it means editing the .kicad_sym.

Prec on the rotary board's R104 goes too; it said "1%", which is now in
that part's entry in Hardware/parts.txt.

Verified by exporting a netlist for each of the seven projects before
and after: every net, and every pin on every net, is identical.

Signed-off-by: Linus Torvalds <torvalds@linux-foundation.org>
Parts:
- D1: LCSC C64898 -> (none)
- R16, R17: JLCPCB C25900 -> (none)
- U2: JLCPCB C130011 -> (none)
- U4: JLCPCB C47122155 -> (none)
- U5: JLCPCB C222104 -> (none)

Commit message: Fill in the manufacturer part numbers from the parts list
Every symbol that carries an LCSC PN now carries the manufacturer's own
part number beside it: 349 of them, against 17 before.  100 went into a
MANUFACTURER_PART_NUMBER field that already existed and was empty, and
232 needed the field creating, hidden, next to the LCSC PN it came
from.  Fifteen already agreed and were left alone.

The values come from Hardware/parts.txt, keyed on LCSC PN, taking the
part number as the last whitespace-separated token of each entry's
manufacturer line - which is what that line's shape means.

Two capacitors said "Samsung CL32B226KAJNNNE", with the maker's name
inside the part-number field; they now say CL32B226KAJNNNE like
everything else.  The manufacturer is not duplicated into the
schematics at all - parts.txt holds it, and the part number identifies
the part on its own.

Four one-off field names go with this, their contents now recorded
properly:

  Manufacturer / Part#  on the rotary board's L101, which is the Murata
                        LQM2MPN1R0MGHL
  Manufacutrer          the typo, on two inductors: DFE201612E-2R2M=P2
  Part                  on five Schottkys, saying "LRC LMBR130T1G"

That last one is worth a second look rather than a straight delete.
JLCPCB ships C191023 as a Guangdong Hottech 1N5819WS, so the schematic
was naming a different manufacturer's equivalent from the one actually
fitted.  The part number recorded here is what gets assembled; the
disagreement is written down in parts.txt next to the entry.

Netlists exported for all seven projects before and after: every net
and every pin on every net unchanged.

Signed-off-by: Linus Torvalds <torvalds@linux-foundation.org>
Parts:
- C1, C10, C2, C9: MANUFACTURER_PART_NUMBER (none) -> GRM21BR71E225KE11L
- C11, C20: MANUFACTURER_PART_NUMBER (none) -> GRM1555C1E151JA01D
- C13, C14, C16, C17, C18, C19, C22, C3, C4, C7, C8: MANUFACTURER_PART_NUMBER (none) -> GCM188R71E105KA64D
- C24, C25, C26, C29: MANUFACTURER_PART_NUMBER (none) -> GRM188R61E106MA73D
- C27, C28, C30, C31, C5: MANUFACTURER_PART_NUMBER (none) -> CL05B104KO5NNNC
- C6: MANUFACTURER_PART_NUMBER (none) -> EEHZA1V470P
- D1: MANUFACTURER_PART_NUMBER (none) -> SM4007PL
- D2: MANUFACTURER_PART_NUMBER (none) -> LTST-C281KGKT
- J4: MANUFACTURER_PART_NUMBER (none) -> AFH05-S12FIA-1H
- R1, R11, R12, R14, R2, R3, R9: MANUFACTURER_PART_NUMBER (none) -> RT0402FRE071KL
- R10, R13, R15, R4, R5, R6, R7, R8: MANUFACTURER_PART_NUMBER (none) -> MCS04020C1004FE000
- R16, R17: MANUFACTURER_PART_NUMBER (none) -> 0402WGF4701TCE
- U1: MANUFACTURER_PART_NUMBER (none) -> TLV76750DRVR
- U2: MANUFACTURER_PART_NUMBER (none) -> OPA2365AIDR
- U3: MANUFACTURER_PART_NUMBER (none) -> TLV76733DRVR
- U4: MANUFACTURER_PART_NUMBER (none) -> TAC5242IRGER
- U5: MANUFACTURER_PART_NUMBER (none) -> M24C64-FMH6TG
