File: Hardware/codec/codec.kicad_sch (KiCad schematic)
At the start: 18 parts, among them J1 BM28B0.6-24DP/2, U1 M24C02-FMH6TG, U2 TAC5112

Commit message: Delete the empty and duplicate schematic fields
Importing parts from SnapEDA and from JLCPCB's library left a pile of
fields behind, and almost none of them ever held anything.  Counting
fields that are *present* makes this look like a naming problem - four
spellings of a manufacturer part number, three of the JLCPCB number -
but counting the ones that are *populated* says something simpler:

  LCSC PN     351 present   349 filled
  LCSC        141 present     1 filled
  LSCS PN      55 present     0 filled
  MP          113 present     0 filled
  MF          113 present     0 filled
  VENDOR      113 present     0 filled
  Field6      126 present     0 filled

So LCSC PN was already the one that mattered, and the rest is debris.
This removes 1964 property blocks: fourteen field names that are empty
on every symbol in every project, plus LCSC and LSCS PN, plus JLCPCB -
which was populated on fifteen symbols and agreed with LCSC PN on all
fifteen.  The one populated LCSC carried the same value as its own
LCSC PN, so nothing is lost.

None of it comes from the symbol libraries: only Reference, Value,
Footprint, Datasheet and Description are defined there, so these do not
grow back when a symbol is updated from its library.  One exception
worth knowing about - a single library symbol does define JLCPCB, so
that one can return, and cleaning it means editing the .kicad_sym.

Prec on the rotary board's R104 goes too; it said "1%", which is now in
that part's entry in Hardware/parts.txt.

Verified by exporting a netlist for each of the seven projects before
and after: every net, and every pin on every net, is identical.

Signed-off-by: Linus Torvalds <torvalds@linux-foundation.org>
Parts:
- R2, R3, R4: JLCPCB C25900 -> (none)
- U1: JLCPCB C222197 -> (none)
Changed lines of the file:
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@@
-			)
-		)
-		(property "JLCPCB" "C222197"
-			(at 151.13 121.92 0)
-			(effects
-				(font
-					(size 1.27 1.27)
-				)
-				(justify right)
-				(hide yes)
 			)
 		)
@@
 			)
 		)
-		(property "JLCPCB" "C25900"
-			(at 212.09 116.84 0)
-			(effects
-				(font
-					(size 1.27 1.27)
-				)
-				(hide yes)
-			)
-		)
 		(property "LCSC PN" "C25900"
 			(at 212.09 116.84 90)
@@
 			)
 		)
-		(property "JLCPCB" "C25900"
-			(at 212.09 113.03 0)
-			(effects
-				(font
-					(size 1.27 1.27)
-				)
-				(hide yes)
-			)
-		)
 		(property "LCSC PN" "C25900"
 			(at 212.09 113.03 90)
@@
 			)
 		)
-		(property "JLCPCB" "C25900"
-			(at 63.5 143.51 0)
-			(effects
-				(font
-					(size 1.27 1.27)
-				)
-				(hide yes)
-			)
-		)
 		(property "LCSC PN" "C25900"
 			(at 63.5 143.51 0)
@@
 			)
 		)
-		(property "Availability" ""
-			(at 209.55 73.66 0)
-			(effects
-				(font
-					(size 1.27 1.27)
-				)
-				(hide yes)
-			)
-		)
-		(property "Check_prices" ""
-			(at 209.55 73.66 0)
-			(effects
-				(font
-					(size 1.27 1.27)
-				)
-				(hide yes)
-			)
-		)
-		(property "Description_1" ""
-			(at 209.55 73.66 0)
-			(effects
-				(font
-					(size 1.27 1.27)
-				)
-				(hide yes)
-			)
-		)
 		(property "MANUFACTURER_PART_NUMBER" ""
 			(at 209.55 73.66 0)
@@
 			)
 		)
-		(property "MF" ""
-			(at 209.55 73.66 0)
-			(effects
-				(font
-					(size 1.27 1.27)
-				)
-				(hide yes)
-			)
-		)
-		(property "MP" ""
-			(at 209.55 73.66 0)
-			(effects
-				(font
-					(size 1.27 1.27)
-				)
-				(hide yes)
-			)
-		)
-		(property "PROD_ID" ""
-			(at 209.55 73.66 0)
-			(effects
-				(font
-					(size 1.27 1.27)
-				)
-				(hide yes)
-			)
-		)
-		(property "Package" ""
-			(at 209.55 73.66 0)
-			(effects
-				(font
-					(size 1.27 1.27)
-				)
-				(hide yes)
-			)
-		)
-		(property "Price" ""
-			(at 209.55 73.66 0)
-			(effects
-				(font
-					(size 1.27 1.27)
-				)
-				(hide yes)
-			)
-		)
 		(property "Sim.Device" ""
 			(at 209.55 73.66 0)
@@
 			(at 209.55 73.66 0)
 			(effects
-				(font
-					(size 1.27 1.27)
-				)
-				(hide yes)
-			)
-		)
-		(property "SnapEDA_Link" ""
-			(at 209.55 73.66 0)
-			(effects
-				(font
-					(size 1.27 1.27)
-				)
-				(hide yes)
-			)
-		)
-		(property "VENDOR" ""
-			(at 209.55 73.66 0)
-			(effects

Commit message: Fill in the manufacturer part numbers from the parts list
Every symbol that carries an LCSC PN now carries the manufacturer's own
part number beside it: 349 of them, against 17 before.  100 went into a
MANUFACTURER_PART_NUMBER field that already existed and was empty, and
232 needed the field creating, hidden, next to the LCSC PN it came
from.  Fifteen already agreed and were left alone.

The values come from Hardware/parts.txt, keyed on LCSC PN, taking the
part number as the last whitespace-separated token of each entry's
manufacturer line - which is what that line's shape means.

Two capacitors said "Samsung CL32B226KAJNNNE", with the maker's name
inside the part-number field; they now say CL32B226KAJNNNE like
everything else.  The manufacturer is not duplicated into the
schematics at all - parts.txt holds it, and the part number identifies
the part on its own.

Four one-off field names go with this, their contents now recorded
properly:

  Manufacturer / Part#  on the rotary board's L101, which is the Murata
                        LQM2MPN1R0MGHL
  Manufacutrer          the typo, on two inductors: DFE201612E-2R2M=P2
  Part                  on five Schottkys, saying "LRC LMBR130T1G"

That last one is worth a second look rather than a straight delete.
JLCPCB ships C191023 as a Guangdong Hottech 1N5819WS, so the schematic
was naming a different manufacturer's equivalent from the one actually
fitted.  The part number recorded here is what gets assembled; the
disagreement is written down in parts.txt next to the entry.

Netlists exported for all seven projects before and after: every net
and every pin on every net unchanged.

Signed-off-by: Linus Torvalds <torvalds@linux-foundation.org>
Parts:
- C1, C2, C3, C6: MANUFACTURER_PART_NUMBER (none) -> GRM188R61E106MA73D
- C10, C4, C5, C7: MANUFACTURER_PART_NUMBER (none) -> CL05B104KO5NNNC
- C8, C9: MANUFACTURER_PART_NUMBER (none) -> CC0603JRX7R7BB105
- D1: MANUFACTURER_PART_NUMBER (none) -> LTST-C281KGKT
- J1: MANUFACTURER_PART_NUMBER (none) -> BM28B0.6-24DP/2-0.35V(51)
- R1: MANUFACTURER_PART_NUMBER (none) -> 0402WGF1001TCE
- R2, R3, R4: MANUFACTURER_PART_NUMBER (none) -> 0402WGF4701TCE
- U1: MANUFACTURER_PART_NUMBER (none) -> M24C02-FMH6TG
- U2: MANUFACTURER_PART_NUMBER (none) -> TAC5112IRGER
Changed lines of the file:
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@@
+			)
+		)
+		(property "MANUFACTURER_PART_NUMBER" "M24C02-FMH6TG"
+			(at 152.4 109.22 0)
+			(hide yes)
+			(show_name no)
+			(do_not_autoplace no)
+			(effects
+				(font
+					(size 1.27 1.27)
+				)
 			)
 		)
@@
 			)
 		)
+		(property "MANUFACTURER_PART_NUMBER" "CL05B104KO5NNNC"
+			(at 100.33 55.88 0)
+			(hide yes)
+			(show_name no)
+			(do_not_autoplace no)
+			(effects
+				(font
+					(size 1.27 1.27)
+				)
+			)
+		)
 		(pin "2"
 		)
@@
 			)
 		)
+		(property "MANUFACTURER_PART_NUMBER" "CC0603JRX7R7BB105"
+			(at 177.8 55.88 0)
+			(hide yes)
+			(show_name no)
+			(do_not_autoplace no)
+			(effects
+				(font
+					(size 1.27 1.27)
+				)
+			)
+		)
 		(pin "2"
 		)
@@
 			)
 		)
+		(property "MANUFACTURER_PART_NUMBER" "GRM188R61E106MA73D"
+			(at 134.62 55.88 0)
+			(hide yes)
+			(show_name no)
+			(do_not_autoplace no)
+			(effects
+				(font
+					(size 1.27 1.27)
+				)
+			)
+		)
 		(pin "2"
 		)
@@
 			)
 		)
+		(property "MANUFACTURER_PART_NUMBER" "LTST-C281KGKT"
+			(at 209.55 82.55 90)
+			(hide yes)
+			(show_name no)
+			(do_not_autoplace no)
+			(effects
+				(font
+					(size 1.27 1.27)
+				)
+			)
+		)
 		(pin "2"
 		)
@@
 			)
 		)
+		(property "MANUFACTURER_PART_NUMBER" "CL05B104KO5NNNC"
+			(at 171.45 121.92 0)
+			(hide yes)
+			(show_name no)
+			(do_not_autoplace no)
+			(effects
+				(font
+					(size 1.27 1.27)
+				)
+			)
+		)
 		(pin "2"
 		)
@@
 			)
 		)
+		(property "MANUFACTURER_PART_NUMBER" "0402WGF4701TCE"
+			(at 212.09 116.84 90)
+			(hide yes)
+			(show_name no)
+			(do_not_autoplace no)
+			(effects
+				(font
+					(size 1.27 1.27)
+				)
+			)
+		)
 		(pin "2"
 		)
@@
 			)
 		)
+		(property "MANUFACTURER_PART_NUMBER" "CL05B104KO5NNNC"
+			(at 86.36 55.88 0)
+			(hide yes)
+			(show_name no)
+			(do_not_autoplace no)
+			(effects
+				(font
+					(size 1.27 1.27)
+				)
+			)
+		)
 		(pin "2"
 		)
@@
 			)
 		)
+		(property "MANUFACTURER_PART_NUMBER" "GRM188R61E106MA73D"
+			(at 72.39 55.88 0)
+			(hide yes)
+			(show_name no)
+			(do_not_autoplace no)
+			(effects
+				(font
+					(size 1.27 1.27)
+				)
+			)
+		)
 		(pin "2"
 		)
@@
 			)
 		)
+		(property "MANUFACTURER_PART_NUMBER" "CC0603JRX7R7BB105"
+			(at 161.29 55.88 0)
+			(hide yes)
+			(show_name no)
+			(do_not_autoplace no)
+			(effects
+				(font
+					(size 1.27 1.27)
+				)
+			)
+		)
 		(pin "2"
 		)
@@
 			)
 		)
+		(property "MANUFACTURER_PART_NUMBER" "GRM188R61E106MA73D"
+			(at 44.45 55.88 0)
+			(hide yes)
+			(show_name no)
+			(do_not_autoplace no)
+			(effects
+				(font
+					(size 1.27 1.27)
+				)
+			)
+		)
 		(pin "2"
 		)
@@
 				)
 				(hide yes)
+			)
+		)
+		(property "MANUFACTURER_PART_NUMBER" "0402WGF4701TCE"
+			(at 212.09 113.03 90)
+			(hide yes)
+			(show_name no)
+			(do_not_autoplace no)
+			(effects
+				(font
+					(size 1.27 1.27)
+				)
 			)
 		)
@@
 			)
 		)
+		(property "MANUFACTURER_PART_NUMBER" "0402WGF4701TCE"
+			(at 63.5 143.51 0)
+			(hide yes)
+			(show_name no)
+			(do_not_autoplace no)
+			(effects
+				(font
+					(size 1.27 1.27)
+				)
+			)
+		)
 		(pin "2"
 		)
@@
 			)
 		)
+		(property "MANUFACTURER_PART_NUMBER" "GRM188R61E106MA73D"
+			(at 58.42 55.88 0)
+			(hide yes)
+			(show_name no)
+			(do_not_autoplace no)
+			(effects
+				(font
+					(size 1.27 1.27)
+				)
+			)
+		)
 		(pin "2"
 		)
@@
 			)
 		)
-		(property "MANUFACTURER_PART_NUMBER" ""
+		(property "MANUFACTURER_PART_NUMBER" "0402WGF1001TCE"
 			(at 209.55 73.66 0)
 			(effects
@@
 			)
 		)
+		(property "MANUFACTURER_PART_NUMBER" "CL05B104KO5NNNC"
+			(at 142.24 55.88 0)
+			(hide yes)
+			(show_name no)
+			(do_not_autoplace no)
+			(effects
+				(font
+					(size 1.27 1.27)
+				)
+			)
+		)
 		(pin "2"
 		)
@@
 			)
 		)
+		(property "MANUFACTURER_PART_NUMBER" "BM28B0.6-24DP/2-0.35V(51)"
+			(at 252.73 80.01 0)
+			(hide yes)
+			(show_name no)
+			(do_not_autoplace no)
+			(effects
+				(font
+					(size 1.27 1.27)
+				)
+			)
+		)
 		(pin "24"
 		)
@@
 			)
 		)
+		(property "MANUFACTURER_PART_NUMBER" "TAC5112IRGER"
+			(at 83.82 115.57 0)
+			(hide yes)
+			(show_name no)
+			(do_not_autoplace no)
+			(effects
+				(font
+					(size 1.27 1.27)
+				)
+			)
+		)
