File: Hardware/rp2354/rp2354.kicad_sch (KiCad schematic)
At the start: 30 parts, among them U1 RP2354A, Y1 ABM8-272-T3

Commit message: Fill in the manufacturer part numbers from the parts list
Every symbol that carries an LCSC PN now carries the manufacturer's own
part number beside it: 349 of them, against 17 before.  100 went into a
MANUFACTURER_PART_NUMBER field that already existed and was empty, and
232 needed the field creating, hidden, next to the LCSC PN it came
from.  Fifteen already agreed and were left alone.

The values come from Hardware/parts.txt, keyed on LCSC PN, taking the
part number as the last whitespace-separated token of each entry's
manufacturer line - which is what that line's shape means.

Two capacitors said "Samsung CL32B226KAJNNNE", with the maker's name
inside the part-number field; they now say CL32B226KAJNNNE like
everything else.  The manufacturer is not duplicated into the
schematics at all - parts.txt holds it, and the part number identifies
the part on its own.

Four one-off field names go with this, their contents now recorded
properly:

  Manufacturer / Part#  on the rotary board's L101, which is the Murata
                        LQM2MPN1R0MGHL
  Manufacutrer          the typo, on two inductors: DFE201612E-2R2M=P2
  Part                  on five Schottkys, saying "LRC LMBR130T1G"

That last one is worth a second look rather than a straight delete.
JLCPCB ships C191023 as a Guangdong Hottech 1N5819WS, so the schematic
was naming a different manufacturer's equivalent from the one actually
fitted.  The part number recorded here is what gets assembled; the
disagreement is written down in parts.txt next to the entry.

Netlists exported for all seven projects before and after: every net
and every pin on every net unchanged.

Signed-off-by: Linus Torvalds <torvalds@linux-foundation.org>
Parts:
- C1, C17, C18, C19, C2, C20, C21, C3, C5: MANUFACTURER_PART_NUMBER (none) -> GRM155R61E475ME15D
- C10, C11, C12, C13, C14, C4, C6, C7, C8, C9: MANUFACTURER_PART_NUMBER (none) -> GRM033Z71C104ME14D
- C15, C16: MANUFACTURER_PART_NUMBER (none) -> GRM0335C1E150JA01D
- L1: MANUFACTURER_PART_NUMBER (none) -> AOTA-B201610S3R3-101-T
- R1, R4, R5: MANUFACTURER_PART_NUMBER (none) -> 0201WMJ0330TEE
- R2, R3, R6: MANUFACTURER_PART_NUMBER (none) -> 0201WMF1001TEE
- U1: MANUFACTURER_PART_NUMBER (none) -> RP2354A
- Y1: MANUFACTURER_PART_NUMBER (none) -> ABM8-272-T3
