File: Hardware/single-input/single-input.kicad_sch (KiCad schematic)
At the start: 32 parts, among them J901 AudioJack3_SwitchTR, U902 OPA2365AIDR, U903 TAC5242

Commit message: Delete the empty and duplicate schematic fields
Importing parts from SnapEDA and from JLCPCB's library left a pile of
fields behind, and almost none of them ever held anything.  Counting
fields that are *present* makes this look like a naming problem - four
spellings of a manufacturer part number, three of the JLCPCB number -
but counting the ones that are *populated* says something simpler:

  LCSC PN     351 present   349 filled
  LCSC        141 present     1 filled
  LSCS PN      55 present     0 filled
  MP          113 present     0 filled
  MF          113 present     0 filled
  VENDOR      113 present     0 filled
  Field6      126 present     0 filled

So LCSC PN was already the one that mattered, and the rest is debris.
This removes 1964 property blocks: fourteen field names that are empty
on every symbol in every project, plus LCSC and LSCS PN, plus JLCPCB -
which was populated on fifteen symbols and agreed with LCSC PN on all
fifteen.  The one populated LCSC carried the same value as its own
LCSC PN, so nothing is lost.

None of it comes from the symbol libraries: only Reference, Value,
Footprint, Datasheet and Description are defined there, so these do not
grow back when a symbol is updated from its library.  One exception
worth knowing about - a single library symbol does define JLCPCB, so
that one can return, and cleaning it means editing the .kicad_sym.

Prec on the rotary board's R104 goes too; it said "1%", which is now in
that part's entry in Hardware/parts.txt.

Verified by exporting a netlist for each of the seven projects before
and after: every net, and every pin on every net, is identical.

Signed-off-by: Linus Torvalds <torvalds@linux-foundation.org>
Parts:
- U903: JLCPCB C47122155 -> (none)

Commit message: Fill in the manufacturer part numbers from the parts list
Every symbol that carries an LCSC PN now carries the manufacturer's own
part number beside it: 349 of them, against 17 before.  100 went into a
MANUFACTURER_PART_NUMBER field that already existed and was empty, and
232 needed the field creating, hidden, next to the LCSC PN it came
from.  Fifteen already agreed and were left alone.

The values come from Hardware/parts.txt, keyed on LCSC PN, taking the
part number as the last whitespace-separated token of each entry's
manufacturer line - which is what that line's shape means.

Two capacitors said "Samsung CL32B226KAJNNNE", with the maker's name
inside the part-number field; they now say CL32B226KAJNNNE like
everything else.  The manufacturer is not duplicated into the
schematics at all - parts.txt holds it, and the part number identifies
the part on its own.

Four one-off field names go with this, their contents now recorded
properly:

  Manufacturer / Part#  on the rotary board's L101, which is the Murata
                        LQM2MPN1R0MGHL
  Manufacutrer          the typo, on two inductors: DFE201612E-2R2M=P2
  Part                  on five Schottkys, saying "LRC LMBR130T1G"

That last one is worth a second look rather than a straight delete.
JLCPCB ships C191023 as a Guangdong Hottech 1N5819WS, so the schematic
was naming a different manufacturer's equivalent from the one actually
fitted.  The part number recorded here is what gets assembled; the
disagreement is written down in parts.txt next to the entry.

Netlists exported for all seven projects before and after: every net
and every pin on every net unchanged.

Signed-off-by: Linus Torvalds <torvalds@linux-foundation.org>
Parts:
- C903, C904, C906, C907, C910, C911, C912, C922, C923: MANUFACTURER_PART_NUMBER (none) -> GRM188Z71E225KE43D
- C905, C918, C919, C921: MANUFACTURER_PART_NUMBER (none) -> GRM033Z71C104ME14D
- C908, C913: MANUFACTURER_PART_NUMBER (none) -> GRM1555C1E151JA01D
- C915, C916, C917, C920: MANUFACTURER_PART_NUMBER (none) -> GRM188R61E106MA73D
- R901, R902, R907, R908: MANUFACTURER_PART_NUMBER (none) -> RT0402BRD07100RL
- R903, R904, R905, R906: MANUFACTURER_PART_NUMBER (none) -> MCS04020C1004FE000
- U902: MANUFACTURER_PART_NUMBER (none) -> OPA2365AIDR
- U903: MANUFACTURER_PART_NUMBER (none) -> TAC5242IRGER
Changed lines of the file:
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@@
 			)
 		)
-		(property "MANUFACTURER_PART_NUMBER" ""
+		(property "MANUFACTURER_PART_NUMBER" "GRM188Z71E225KE43D"
 			(at 49.53 100.33 0)
 			(hide yes)
@@
 			)
 		)
+		(property "MANUFACTURER_PART_NUMBER" "GRM188Z71E225KE43D"
+			(at 181.61 114.3 0)
+			(hide yes)
+			(show_name no)
+			(do_not_autoplace no)
+			(effects
+				(font
+					(size 1.27 1.27)
+				)
+			)
+		)
 		(property "Sim.Params" ""
 			(at 181.61 114.3 0)
@@
 			)
 		)
-		(property "MANUFACTURER_PART_NUMBER" ""
+		(property "MANUFACTURER_PART_NUMBER" "GRM1555C1E151JA01D"
 			(at 83.82 121.92 0)
 			(hide yes)
@@
 			)
 		)
-		(property "MANUFACTURER_PART_NUMBER" ""
+		(property "MANUFACTURER_PART_NUMBER" "GRM188Z71E225KE43D"
 			(at 135.89 76.2 0)
 			(hide yes)
@@
 			)
 		)
-		(property "MANUFACTURER_PART_NUMBER" ""
+		(property "MANUFACTURER_PART_NUMBER" "MCS04020C1004FE000"
 			(at 38.1 100.33 0)
 			(hide yes)
@@
 			)
 		)
+		(property "MANUFACTURER_PART_NUMBER" "GRM188R61E106MA73D"
+			(at 181.61 45.72 0)
+			(hide yes)
+			(show_name no)
+			(do_not_autoplace no)
+			(effects
+				(font
+					(size 1.27 1.27)
+				)
+			)
+		)
 		(property "Sim.Params" ""
 			(at 181.61 45.72 0)
@@
 			)
 		)
-		(property "MANUFACTURER_PART_NUMBER" ""
+		(property "MANUFACTURER_PART_NUMBER" "GRM188Z71E225KE43D"
 			(at 135.89 86.36 0)
 			(hide yes)
@@
 			)
 		)
-		(property "MANUFACTURER_PART_NUMBER" ""
+		(property "MANUFACTURER_PART_NUMBER" "RT0402BRD07100RL"
 			(at 74.93 73.66 0)
 			(hide yes)
@@
 			)
 		)
+		(property "MANUFACTURER_PART_NUMBER" "GRM188R61E106MA73D"
+			(at 181.61 71.12 0)
+			(hide yes)
+			(show_name no)
+			(do_not_autoplace no)
+			(effects
+				(font
+					(size 1.27 1.27)
+				)
+			)
+		)
 		(property "Sim.Params" ""
 			(at 181.61 71.12 0)
@@
 			)
 		)
-		(property "MANUFACTURER_PART_NUMBER" ""
+		(property "MANUFACTURER_PART_NUMBER" "GRM1555C1E151JA01D"
 			(at 83.82 81.28 0)
 			(hide yes)
@@
 			)
 		)
-		(property "MANUFACTURER_PART_NUMBER" ""
+		(property "MANUFACTURER_PART_NUMBER" "MCS04020C1004FE000"
 			(at 38.1 90.17 0)
 			(hide yes)
@@
 			)
 		)
+		(property "MANUFACTURER_PART_NUMBER" "GRM188Z71E225KE43D"
+			(at 181.61 92.71 0)
+			(hide yes)
+			(show_name no)
+			(do_not_autoplace no)
+			(effects
+				(font
+					(size 1.27 1.27)
+				)
+			)
+		)
 		(property "Sim.Params" ""
 			(at 181.61 92.71 0)
@@
 			)
 		)
-		(property "MANUFACTURER_PART_NUMBER" ""
+		(property "MANUFACTURER_PART_NUMBER" "MCS04020C1004FE000"
 			(at 67.31 86.36 0)
 			(hide yes)
@@
 			)
 		)
-		(property "MANUFACTURER_PART_NUMBER" ""
+		(property "MANUFACTURER_PART_NUMBER" "RT0402BRD07100RL"
 			(at 74.93 114.3 0)
 			(hide yes)
@@
 			)
 		)
+		(property "MANUFACTURER_PART_NUMBER" "GRM033Z71C104ME14D"
+			(at 237.49 45.72 0)
+			(hide yes)
+			(show_name no)
+			(do_not_autoplace no)
+			(effects
+				(font
+					(size 1.27 1.27)
+				)
+			)
+		)
 		(property "Sim.Params" ""
 			(at 237.49 45.72 0)
@@
 			)
 		)
+		(property "MANUFACTURER_PART_NUMBER" "OPA2365AIDR"
+			(at 96.52 41.91 0)
+			(hide yes)
+			(show_name no)
+			(do_not_autoplace no)
+			(effects
+				(font
+					(size 1.27 1.27)
+				)
+			)
+		)
 		(pin "4"
 		)
@@
 			)
 		)
+		(property "MANUFACTURER_PART_NUMBER" "GRM033Z71C104ME14D"
+			(at 223.52 45.72 0)
+			(hide yes)
+			(show_name no)
+			(do_not_autoplace no)
+			(effects
+				(font
+					(size 1.27 1.27)
+				)
+			)
+		)
 		(property "Sim.Params" ""
 			(at 223.52 45.72 0)
@@
 			)
 		)
+		(property "MANUFACTURER_PART_NUMBER" "GRM033Z71C104ME14D"
+			(at 189.23 71.12 0)
+			(hide yes)
+			(show_name no)
+			(do_not_autoplace no)
+			(effects
+				(font
+					(size 1.27 1.27)
+				)
+			)
+		)
 		(property "Sim.Params" ""
 			(at 189.23 71.12 0)
@@
 			)
 		)
-		(property "MANUFACTURER_PART_NUMBER" ""
+		(property "MANUFACTURER_PART_NUMBER" "GRM188Z71E225KE43D"
 			(at 135.89 116.84 0)
 			(hide yes)
@@
 			)
 		)
+		(property "MANUFACTURER_PART_NUMBER" "OPA2365AIDR"
+			(at 99.06 116.84 0)
+			(hide yes)
+			(show_name no)
+			(do_not_autoplace no)
+			(effects
+				(font
+					(size 1.27 1.27)
+				)
+			)
+		)
 		(pin "4"
 		)
@@
 			)
 		)
+		(property "MANUFACTURER_PART_NUMBER" "OPA2365AIDR"
+			(at 99.06 76.2 0)
+			(hide yes)
+			(show_name no)
+			(do_not_autoplace no)
+			(effects
+				(font
+					(size 1.27 1.27)
+				)
+			)
+		)
 		(pin "4"
 		)
@@
 			)
 		)
-		(property "MANUFACTURER_PART_NUMBER" ""
+		(property "MANUFACTURER_PART_NUMBER" "RT0402BRD07100RL"
 			(at 118.11 116.84 0)
 			(hide yes)
@@
 			)
 		)
-		(property "MANUFACTURER_PART_NUMBER" ""
+		(property "MANUFACTURER_PART_NUMBER" "GRM188Z71E225KE43D"
 			(at 59.69 73.66 0)
 			(hide yes)
@@
 			)
 		)
-		(property "MANUFACTURER_PART_NUMBER" ""
+		(property "MANUFACTURER_PART_NUMBER" "GRM188Z71E225KE43D"
 			(at 59.69 114.3 0)
 			(hide yes)
@@
 			)
 		)
-		(property "MANUFACTURER_PART_NUMBER" ""
+		(property "MANUFACTURER_PART_NUMBER" "GRM033Z71C104ME14D"
 			(at 78.74 41.91 0)
 			(hide yes)
@@
 			)
 		)
+		(property "MANUFACTURER_PART_NUMBER" "GRM188R61E106MA73D"
+			(at 209.55 45.72 0)
+			(hide yes)
+			(show_name no)
+			(do_not_autoplace no)
+			(effects
+				(font
+					(size 1.27 1.27)
+				)
+			)
+		)
 		(property "Sim.Params" ""
 			(at 209.55 45.72 0)
@@
 			)
 		)
-		(property "MANUFACTURER_PART_NUMBER" ""
+		(property "MANUFACTURER_PART_NUMBER" "MCS04020C1004FE000"
 			(at 67.31 104.14 0)
 			(hide yes)
@@
 			)
 		)
-		(property "MANUFACTURER_PART_NUMBER" ""
+		(property "MANUFACTURER_PART_NUMBER" "RT0402BRD07100RL"
 			(at 118.11 76.2 0)
 			(hide yes)
@@
 			)
 		)
+		(property "MANUFACTURER_PART_NUMBER" "GRM188R61E106MA73D"
+			(at 195.58 45.72 0)
+			(hide yes)
+			(show_name no)
+			(do_not_autoplace no)
+			(effects
+				(font
+					(size 1.27 1.27)
+				)
+			)
+		)
 		(property "Sim.Params" ""
 			(at 195.58 45.72 0)
@@
 			)
 		)
+		(property "MANUFACTURER_PART_NUMBER" "TAC5242IRGER"
+			(at 240.03 100.33 0)
+			(hide yes)
+			(show_name no)
+			(do_not_autoplace no)
+			(effects
+				(font
+					(size 1.27 1.27)
+				)
+			)
+		)
 		(property "Sim.Params" ""
 			(at 240.03 100.33 0)
@@
 			)
 		)
-		(property "MANUFACTURER_PART_NUMBER" ""
+		(property "MANUFACTURER_PART_NUMBER" "GRM188Z71E225KE43D"
 			(at 135.89 127 0)
 			(hide yes)
