File: Hardware/usb-stomp/rp2354.kicad_sch (KiCad schematic)
At the start: 30 parts, among them U401 RP2354A, Y401 ABM8-272-T3

Commit message: Let's re-do the usb-stomp board without the flex board
It was a teaching experience, but I guess the lesson was "don't do
that".  Let's just turn it into a straightforward simple single board.

I did decide to try a buck regulator, and I'm also playing with adding
support for a remote stomp switch or expression pedal.  I'm trying to do
it in a way that pretty much anything could be made to work - a single
remote stomp over a TS 1/4" cable, or a dual remote stomp over a TRS
one.  Or an expression pedal. But maybe I screwed that thing up.

The TRS Typa-A midi ports remain for remote control, but I'm thinking
that it shouldn't be too hard to teach WebMIDI to set up a model where
the remote stomp / expression pedal can control some arbitrary pot
value in the scene.

There's also a rotary encoder for the same reason - program the scene to
make it be the master volume, or the noise gate level, or whatever.

Of course, that "program the scene" part is all just a nebulous plan.  I
don't actually support that yet.  SMOP.

Signed-off-by: Linus Torvalds <torvalds@linux-foundation.org>
Other:
- moved on the sheet: C401, C402, C403, C404, C405, C406, C407, C408, C409, C410, C411, C412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

Commit message: Fill in the manufacturer part numbers from the parts list
Every symbol that carries an LCSC PN now carries the manufacturer's own
part number beside it: 349 of them, against 17 before.  100 went into a
MANUFACTURER_PART_NUMBER field that already existed and was empty, and
232 needed the field creating, hidden, next to the LCSC PN it came
from.  Fifteen already agreed and were left alone.

The values come from Hardware/parts.txt, keyed on LCSC PN, taking the
part number as the last whitespace-separated token of each entry's
manufacturer line - which is what that line's shape means.

Two capacitors said "Samsung CL32B226KAJNNNE", with the maker's name
inside the part-number field; they now say CL32B226KAJNNNE like
everything else.  The manufacturer is not duplicated into the
schematics at all - parts.txt holds it, and the part number identifies
the part on its own.

Four one-off field names go with this, their contents now recorded
properly:

  Manufacturer / Part#  on the rotary board's L101, which is the Murata
                        LQM2MPN1R0MGHL
  Manufacutrer          the typo, on two inductors: DFE201612E-2R2M=P2
  Part                  on five Schottkys, saying "LRC LMBR130T1G"

That last one is worth a second look rather than a straight delete.
JLCPCB ships C191023 as a Guangdong Hottech 1N5819WS, so the schematic
was naming a different manufacturer's equivalent from the one actually
fitted.  The part number recorded here is what gets assembled; the
disagreement is written down in parts.txt next to the entry.

Netlists exported for all seven projects before and after: every net
and every pin on every net unchanged.

Signed-off-by: Linus Torvalds <torvalds@linux-foundation.org>
Parts:
- C401, C402, C403, C405, C413, C415, C417, C420, C421: MANUFACTURER_PART_NUMBER (none) -> GRM155R61E475ME15D
- C404, C406, C407, C408, C409, C410, C411, C412, C414, C416: MANUFACTURER_PART_NUMBER (none) -> GRM033Z71C104ME14D
- C418, C419: MANUFACTURER_PART_NUMBER (none) -> GRM0335C1E150JA01D
- L401: MANUFACTURER_PART_NUMBER (none) -> AOTA-B201610S3R3-101-T
- R401, R404, R405: MANUFACTURER_PART_NUMBER (none) -> 0201WMJ0330TEE
- R402, R403, R406: MANUFACTURER_PART_NUMBER (none) -> 0201WMF1001TEE
- U401: MANUFACTURER_PART_NUMBER (none) -> RP2354A
- Y401: MANUFACTURER_PART_NUMBER (none) -> ABM8-272-T3
