File: Hardware/usb-stomp/rp2354.kicad_sch (KiCad schematic)
At the start: 30 parts, among them U401 RP2354A, Y401 ABM8-272-T3

Commit message: Update the usb-stomp parts selection in the schematic
This updates the 0201 parts to 0402 sizes, because the 0201 sizing was
just inconvenient and caused problems with the (failed) flex board trial
too.  The board has plenty of space, the 0201 sizing was to make it
easier to route all the traces out of the RP2354, but it's not like I
use all the GPIOs anyway.

So let's re-route for a saner component choice.

The actual noticeable change comes from also picking a larger 4.7uF
capacitor on the input path to help improve the bass response into the
codec further. The -3 dB point should now be below 10Hz.

The actual PCB changes next.

Signed-off-by: Linus Torvalds <torvalds@linux-foundation.org>
Parts:
- C404, C406, C407, C408, C409, C410, C411, C412, C414, C416: footprint Capacitor_SMD:C_0201_0603Metric -> Capacitor_SMD:C_0402_1005Metric; LCSC PN C3901090 -> C1525; MANUFACTURER_PART_NUMBER GRM033Z71C104ME14D -> CL05B104KO5NNNC
- C418, C419: footprint Capacitor_SMD:C_0201_0603Metric -> Capacitor_SMD:C_0402_1005Metric; LCSC PN C161373 -> C76950; MANUFACTURER_PART_NUMBER GRM0335C1E150JA01D -> GRM1555C1H150JA01D
- R401, R404, R405: value 33R -> 33Ω; footprint Resistor_SMD:R_0201_0603Metric -> Resistor_SMD:R_0402_1005Metric; LCSC PN C423356 -> C25105; MANUFACTURER_PART_NUMBER 0201WMJ0330TEE -> 0402WGF330JTCE
- R402, R403, R406: value 1k -> 1kΩ; footprint Resistor_SMD:R_0201_0603Metric -> Resistor_SMD:R_0402_1005Metric; LCSC PN C270365 -> C11702; MANUFACTURER_PART_NUMBER 0201WMF1001TEE -> 0402WGF1001TCE
