File: Hardware/usb-stomp/tac5242.kicad_sch (KiCad schematic)
At the start: 35 parts, among them J301 AudioJack3_SwitchTR, U103 TLV76733DRVx, U301 OPA2365AIDR, U302 TAC5242

Commit message: Let's re-do the usb-stomp board without the flex board
It was a teaching experience, but I guess the lesson was "don't do
that".  Let's just turn it into a straightforward simple single board.

I did decide to try a buck regulator, and I'm also playing with adding
support for a remote stomp switch or expression pedal.  I'm trying to do
it in a way that pretty much anything could be made to work - a single
remote stomp over a TS 1/4" cable, or a dual remote stomp over a TRS
one.  Or an expression pedal. But maybe I screwed that thing up.

The TRS Typa-A midi ports remain for remote control, but I'm thinking
that it shouldn't be too hard to teach WebMIDI to set up a model where
the remote stomp / expression pedal can control some arbitrary pot
value in the scene.

There's also a rotary encoder for the same reason - program the scene to
make it be the master volume, or the noise gate level, or whatever.

Of course, that "program the scene" part is all just a nebulous plan.  I
don't actually support that yet.  SMOP.

Signed-off-by: Linus Torvalds <torvalds@linux-foundation.org>
Parts:
- removed C126: 2.2uF, Capacitor_SMD:C_0603_1608Metric, symbol Device:C
- added C304, C309: 2.2nF, Capacitor_SMD:C_0402_1005Metric, symbol Device:C
- added C305, C310: 2.2uF, Capacitor_SMD:C_0603_1608Metric, symbol Device:C
- added C317: 22uF, Capacitor_SMD:C_1210_3225Metric, symbol Device:C
- added J301: AudioJack3_SwitchTR, Mylib:NRJ6HM-1-PRE, symbol Connector_Audio:AudioJack3_SwitchTR
- added L301: 2.2uH, Mylib:L_0806, symbol Device:L
- added R303, R309: 1k, Resistor_SMD:R_0402_1005Metric, symbol Device:R
- added R306, R310: 1MEG, Resistor_SMD:R_0402_1005Metric, symbol Device:R
- added R313: 1R, Resistor_SMD:R_0402_1005Metric, symbol Device:R
- renumbered C304 to C306, C305 to C307, C306 to C308, C307 to C311, C308 to C312, C309 to C313, C310 to C314, C311 to C315, C312 to C316, C127 to C318, C313 to C319, C314 to C320, C315 to C321, C316 to C322, C317 to C323, C318 to C324, C319 to C325, C320 to C326, C321 to C327, J301 to J302, R303 to R304, R304 to R305, R305 to R307, R306 to R308, R307 to R311, R308 to R312, U103 to U302, U302 to U303
Connections:
- net +5V: now also L301.1, R313.1; no longer U302.6 (IN)
- net GND: now also C304.1, C309.1, C317.2, J301.S, R306.2, R310.2
- net OUT1P: now also R303.1
- net OUT2P: now also R309.1
- new net: C304.2, C305.1, R303.2
- new net: C309.2, C310.1, R309.2
- new net: C317.1, L301.2, R313.2, U302.6 (IN)
- new net OUT^{LEFT}: C305.2, J301.T, R306.1
- new net OUT^{RIGHT}: C310.2, J301.R, R310.1
- no-connect marks 4 -> 6
Other:
- moved on the sheet: C318, U302

Commit message: Delete the empty and duplicate schematic fields
Importing parts from SnapEDA and from JLCPCB's library left a pile of
fields behind, and almost none of them ever held anything.  Counting
fields that are *present* makes this look like a naming problem - four
spellings of a manufacturer part number, three of the JLCPCB number -
but counting the ones that are *populated* says something simpler:

  LCSC PN     351 present   349 filled
  LCSC        141 present     1 filled
  LSCS PN      55 present     0 filled
  MP          113 present     0 filled
  MF          113 present     0 filled
  VENDOR      113 present     0 filled
  Field6      126 present     0 filled

So LCSC PN was already the one that mattered, and the rest is debris.
This removes 1964 property blocks: fourteen field names that are empty
on every symbol in every project, plus LCSC and LSCS PN, plus JLCPCB -
which was populated on fifteen symbols and agreed with LCSC PN on all
fifteen.  The one populated LCSC carried the same value as its own
LCSC PN, so nothing is lost.

None of it comes from the symbol libraries: only Reference, Value,
Footprint, Datasheet and Description are defined there, so these do not
grow back when a symbol is updated from its library.  One exception
worth knowing about - a single library symbol does define JLCPCB, so
that one can return, and cleaning it means editing the .kicad_sym.

Prec on the rotary board's R104 goes too; it said "1%", which is now in
that part's entry in Hardware/parts.txt.

Verified by exporting a netlist for each of the seven projects before
and after: every net, and every pin on every net, is identical.

Signed-off-by: Linus Torvalds <torvalds@linux-foundation.org>
Parts:
- U303: JLCPCB C47122155 -> (none)

Commit message: Fill in the manufacturer part numbers from the parts list
Every symbol that carries an LCSC PN now carries the manufacturer's own
part number beside it: 349 of them, against 17 before.  100 went into a
MANUFACTURER_PART_NUMBER field that already existed and was empty, and
232 needed the field creating, hidden, next to the LCSC PN it came
from.  Fifteen already agreed and were left alone.

The values come from Hardware/parts.txt, keyed on LCSC PN, taking the
part number as the last whitespace-separated token of each entry's
manufacturer line - which is what that line's shape means.

Two capacitors said "Samsung CL32B226KAJNNNE", with the maker's name
inside the part-number field; they now say CL32B226KAJNNNE like
everything else.  The manufacturer is not duplicated into the
schematics at all - parts.txt holds it, and the part number identifies
the part on its own.

Four one-off field names go with this, their contents now recorded
properly:

  Manufacturer / Part#  on the rotary board's L101, which is the Murata
                        LQM2MPN1R0MGHL
  Manufacutrer          the typo, on two inductors: DFE201612E-2R2M=P2
  Part                  on five Schottkys, saying "LRC LMBR130T1G"

That last one is worth a second look rather than a straight delete.
JLCPCB ships C191023 as a Guangdong Hottech 1N5819WS, so the schematic
was naming a different manufacturer's equivalent from the one actually
fitted.  The part number recorded here is what gets assembled; the
disagreement is written down in parts.txt next to the entry.

Netlists exported for all seven projects before and after: every net
and every pin on every net unchanged.

Signed-off-by: Linus Torvalds <torvalds@linux-foundation.org>
Parts:
- C301, C302, C303, C305, C310, C313, C314, C315, C316, C318, C321, C322: MANUFACTURER_PART_NUMBER (none) -> GRM188Z71E225KE43D
- C306, C323, C326, C327: MANUFACTURER_PART_NUMBER (none) -> GRM033Z71C104ME14D
- C307, C308: MANUFACTURER_PART_NUMBER (none) -> GRM1555C1E151JA01D
- C317: MANUFACTURER_PART_NUMBER Samsung CL32B226KAJNNNE -> CL32B226KAJNNNE
- C319, C320, C324, C325: MANUFACTURER_PART_NUMBER (none) -> GRM188R61E106MA73D
- L301: MANUFACTURER_PART_NUMBER (none) -> DFE201612E-2R2M=P2; Manufacutrer Murata DFE201612E-2R2M=P2 -> (none)
- R301, R302, R304, R305, R306, R310: MANUFACTURER_PART_NUMBER (none) -> MCS04020C1004FE000
- R303, R309: MANUFACTURER_PART_NUMBER (none) -> RT0402FRE071KL
- R307, R308, R311, R312: MANUFACTURER_PART_NUMBER (none) -> RT0402BRD07100RL
- R313: MANUFACTURER_PART_NUMBER (none) -> FRC0402F1R00TS
- U301: MANUFACTURER_PART_NUMBER (none) -> OPA2365AIDR
- U302: MANUFACTURER_PART_NUMBER (none) -> TLV76733DRVR
- U303: MANUFACTURER_PART_NUMBER (none) -> TAC5242IRGER
