File: Hardware/usb-stomp/usb-stomp.kicad_sch (KiCad schematic)
At the start: 38 parts, among them J101 USB_C_Receptacle_USB2.0_16P, J102 Barrel_Jack_Switch, J103 AudioJack3_SwitchTR, SW101 SW_SPST, SW102 RotaryEncoder_Switch_MP, U101 USBLC6-2P6, U102 M24C64-FMH6TG, U103 TPS62153, U104 TLV76733DRVx

Commit message: Delete the empty and duplicate schematic fields
Importing parts from SnapEDA and from JLCPCB's library left a pile of
fields behind, and almost none of them ever held anything.  Counting
fields that are *present* makes this look like a naming problem - four
spellings of a manufacturer part number, three of the JLCPCB number -
but counting the ones that are *populated* says something simpler:

  LCSC PN     351 present   349 filled
  LCSC        141 present     1 filled
  LSCS PN      55 present     0 filled
  MP          113 present     0 filled
  MF          113 present     0 filled
  VENDOR      113 present     0 filled
  Field6      126 present     0 filled

So LCSC PN was already the one that mattered, and the rest is debris.
This removes 1964 property blocks: fourteen field names that are empty
on every symbol in every project, plus LCSC and LSCS PN, plus JLCPCB -
which was populated on fifteen symbols and agreed with LCSC PN on all
fifteen.  The one populated LCSC carried the same value as its own
LCSC PN, so nothing is lost.

None of it comes from the symbol libraries: only Reference, Value,
Footprint, Datasheet and Description are defined there, so these do not
grow back when a symbol is updated from its library.  One exception
worth knowing about - a single library symbol does define JLCPCB, so
that one can return, and cleaning it means editing the .kicad_sym.

Prec on the rotary board's R104 goes too; it said "1%", which is now in
that part's entry in Hardware/parts.txt.

Verified by exporting a netlist for each of the seven projects before
and after: every net, and every pin on every net, is identical.

Signed-off-by: Linus Torvalds <torvalds@linux-foundation.org>
Parts:
- U102: JLCPCB C222104 -> (none)

Commit message: Fill in the manufacturer part numbers from the parts list
Every symbol that carries an LCSC PN now carries the manufacturer's own
part number beside it: 349 of them, against 17 before.  100 went into a
MANUFACTURER_PART_NUMBER field that already existed and was empty, and
232 needed the field creating, hidden, next to the LCSC PN it came
from.  Fifteen already agreed and were left alone.

The values come from Hardware/parts.txt, keyed on LCSC PN, taking the
part number as the last whitespace-separated token of each entry's
manufacturer line - which is what that line's shape means.

Two capacitors said "Samsung CL32B226KAJNNNE", with the maker's name
inside the part-number field; they now say CL32B226KAJNNNE like
everything else.  The manufacturer is not duplicated into the
schematics at all - parts.txt holds it, and the part number identifies
the part on its own.

Four one-off field names go with this, their contents now recorded
properly:

  Manufacturer / Part#  on the rotary board's L101, which is the Murata
                        LQM2MPN1R0MGHL
  Manufacutrer          the typo, on two inductors: DFE201612E-2R2M=P2
  Part                  on five Schottkys, saying "LRC LMBR130T1G"

That last one is worth a second look rather than a straight delete.
JLCPCB ships C191023 as a Guangdong Hottech 1N5819WS, so the schematic
was naming a different manufacturer's equivalent from the one actually
fitted.  The part number recorded here is what gets assembled; the
disagreement is written down in parts.txt next to the entry.

Netlists exported for all seven projects before and after: every net
and every pin on every net unchanged.

Signed-off-by: Linus Torvalds <torvalds@linux-foundation.org>
Parts:
- C101, C103, C111: MANUFACTURER_PART_NUMBER (none) -> GRM033Z71C104ME14D
- C102, C104: MANUFACTURER_PART_NUMBER (none) -> GRM188R61E106MA73D
- C105, C108: MANUFACTURER_PART_NUMBER (none) -> 0402B223K500NT
- C106: MANUFACTURER_PART_NUMBER Samsung CL32B226KAJNNNE -> CL32B226KAJNNNE
- C109, C110, C112: MANUFACTURER_PART_NUMBER (none) -> GRM188Z71E225KE43D
- D101, D103, D104, D106: MANUFACTURER_PART_NUMBER (none) -> 1N5819WS; Part LRC LMBR130T1G -> (none)
- D102: MANUFACTURER_PART_NUMBER (none) -> LTST-C281KGKT
- D105, D107: MANUFACTURER_PART_NUMBER (none) -> BAT54SW
- J101: MANUFACTURER_PART_NUMBER (none) -> GT-USB-7010C
- L101: MANUFACTURER_PART_NUMBER (none) -> DFE201612E-2R2M=P2; Manufacutrer Murata DFE201612E-2R2M=P2 -> (none)
- R101, R102, R104, R105: MANUFACTURER_PART_NUMBER (none) -> 0402WGF5101TCE
- R103, R106, R107, R109: MANUFACTURER_PART_NUMBER (none) -> RT0402FRE071KL
- R108: MANUFACTURER_PART_NUMBER (none) -> 0402WGF1003TCE
- U101: MANUFACTURER_PART_NUMBER (none) -> USBLC6-2P6
- U102: MANUFACTURER_PART_NUMBER (none) -> M24C64-FMH6TG
- U103: MANUFACTURER_PART_NUMBER (none) -> TPS62153RGTR
- U104: MANUFACTURER_PART_NUMBER (none) -> TLV76733DRVR
