File: Hardware/pedal/rp2354.kicad_sch (KiCad schematic)
At the start: 30 parts, among them U401 RP2354A, Y401 ABM8-272-T3

Commit message: Create a new board version with 8MB PSRAM and dual stomp switches
This adds a 8MB of external memory to the RP2354.  It's worth noting
that such memory is much slower than the internal SRAM, so while the
intended use is very much for audio effects to store more audio state
(for a looper or a longer echo), it needs to be treated carefully.

The PSRAM _can_ be accessed as just regular memory, exactly the same way
the flash works (it's all using the same QSPI interface).

But the preferred model will be to use a DMA engine to move the data
asynchronously between the on-die SRAM and the off-chip PSRAM, so that
the audio engine running on core 1 will not see random delay states from
the QSPI accesses.

The second stomp switch is partly to make it easier to control any
looper interface, but partly because this pedal really did want two
stomp switches for controlling: you might use one for bypass, and the
other to switch between scenes.

A remote stomp obviously would also work, but let's make really basic
functionality available on the pedal directly.

Note that this will also require a new board file: the GPIO mappings
have changed to make the PCB routing simpler.  I wanted to use GPIO0 for
the new PSRAM QSPI chip select line, because it's right there in that
corner of the RP2354A chip.  But we used to use it for the stomp switch.

And once I changed one GPIO mapping, I might as well change the others,
since a board update is a board update, and the old routing was odd for
historical reasons, going all the way back to how the i2s lines went
over the BM28 connectors and the FFC cable.

So now the GPIO mappings are

 GPIO0: PSRAM QSPI CS1n (didn't exist before)
 GPIO8/9: MIDI UART TX/RX (used to be  20/21)
 GPIO10/19: STOMP 0/1 (used to be GPIO0 for STOMP0)
 GPIO11: WS2812B chain (used to be GPIO25)
 GPIO12..14: rotary encoder A/B/SW (stays the same)
 GPIO20..23: i2s DIN/DOUT/FSYNC/BCLK (used to be 10/11/9/8)

 ADC0/1: expression pedal Tip and Ring (used to be other way ar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
Parts:
- added C404: 0.1uF, Capacitor_SMD:C_0402_1005Metric, symbol Device:C
- added R401: 2.2kΩ, Resistor_SMD:R_0402_1005Metric, symbol Device:R
- added U401: APS6404L-3SQRx-ZR, Package_SON:Winbond_USON-8-1EP_3x2mm_P0.5mm_EP0.2x1.6mm, symbol Memory_RAM:APS6404L-3SQRx-ZR
- R403: renamed from R402; value 1kΩ -> 2.2kΩ; LCSC PN C11702 -> C25879; MANUFACTURER_PART_NUMBER 0402WGF1001TCE -> 0402WGF2201TCE
- renumbered C404 to C405, C405 to C406, C406 to C407, C407 to C408, C408 to C409, C409 to C410, C410 to C411, C411 to C412, C412 to C413, C413 to C414, C414 to C415, C415 to C416, C416 to C417, C417 to C418, C418 to C419, C419 to C420, C420 to C421, C421 to C422, R401 to R402, R403 to R404, R404 to R405, R405 to R406, R406 to R407, U401 to U402
Connections:
- net +3V3: now also C404.1, R401.2, U401.8 (VDD)
- net GND: now also C404.2, U401.4 (VSS), U401.9 (EPAD)
- net GPIO0: now also R401.1, U401.1 (~{CE})
- net SD3: now reaches U402.55 (QSPI_SD3)
- net SD3: now also U401.7 (SIO3)
- net SCLK: now reaches U402.56 (QSPI_SCLK)
- net SCLK: now also U401.6 (SCLK)
- net SD0: now reaches U402.57 (QSPI_SD0)
- net SD0: now also U401.5 (SI/SIO0)
- net SD2: now reaches U402.58 (QSPI_SD2)
- net SD2: now also U401.3 (SIO2)
- net SD1: now reaches U402.59 (QSPI_SD1)
- net SD1: now also U401.2 (SO/SIO1)
- no-connect marks 5 -> 0
