File: Hardware/pedal/pedal.kicad_pcb (KiCad board)
At the start: 4 copper layers, 90 x 70 mm, 134 parts, among them J101 USB_C_Receptacle_USB2.0_16P, J102 Barrel_Jack_Switch, J103 AudioJack3_SwitchTR, J201 AudioJack4, J202 AudioJack4, J301 AudioJack3_SwitchTR, J302 AudioJack3_SwitchTR, SW101 SW_SPST, SW102 SW_SPST, SW103 RotaryEncoder_Switch_MP, U101 USBLC6-2P6, U102 TPS62153, U103 TLV76733DRVx, U201 SN74AHCT1G125DCKR, U202 TLP2310, U301 OPA2365AIDR, U302 TLV76733DRVx, U303 TAC5242, U401 APS6404L-3SQRx-ZR, U402 RP2354A, Y401 ABM8-272-T3

Commit message: Create a new rotary encoder footprint
The standard kicad footprint has long driven me mad.  It's centered on
pin 1, because of whatever insane reasons.  But the location of pin 1 on
a rotary is completely pointless and wrong: the only actual location
that matters is the location of the _shaft_ of the rotary.  That's the
one you want to place.

And this annoyance came to a head when the vendor 3D model I found is sane.

So the insane kicad footprint goes out the window, replaced by something
that actually makes sense.  And associated with a vendor 3D model with
the sensible placement too.

The pedal design has been updated and now the 3D view shows it in all
its proper glory.

Except for the stomp switch. Which I'm afraid I will have to model myself.

It's going to be ugly.  You have been warned.  And the ugliness is only
going to be accentuated by all the much prettier models that will
surround it.  Too bad.

Signed-off-by: Linus Torvalds <torvalds@linux-foundation.org>
Parts:
- SW103: footprint Rotary_Encoder:RotaryEncoder_Alps_EC11E-Switch_Vertical_H20mm -> Mylib:RotaryEncoder_EC11-Switch_Vertical_H20mm
- moved SW103 7.91 mm to (100.0, 105.2)
