File: Hardware/minimal/tac5242.kicad_sch (KiCad schematic)
At the start: 37 parts, among them J301 AudioJack3_SwitchTR, J302 AudioJack3_SwitchTR, U301 OPA2323, U302 TAC5242

Commit message: Commit DC-coupled TAC5112 design
This is a slightly modified 'minimal' board with the same board outline
but an added 3.5mm DC jack.

The upside: no coupling capacitors into the codec that have distortion
at low-end frequencies due to the capacitors' voltage coefficients.  The
existing 0805 4.7uF caps were large for this minimal board, and caused
the THD+N to go to roughly -65dB for a low-B bass signal at a reasonable
signal level of 0.1Vrms.  That's not horrible, but it's not optimal.

The 10Hz corner also caused issues for using the pedal as a measurement
instrument, since it introduced a consistent measurement error that was
initially incorrectly attributed to the pedal under test.

The other upside is simply the existence of the headphone jack.  That
user-visible addition is likely a lot more noticeable than the
low-frequency THD+N improvement this should bring or the improvement in
low-end frequency response.

Downside: the TAC212 with a better noise floor is out of stock, and so I
am back to the slightly lower dynamic range of the TAC5112 - but with
the new fixed footprint with proper paste and thermal vias.  The thermal
pad is likely to actually come into play now that the codec is used as a
headphone amplifier too.

The lower dynamic range is unlikely to be noticeable - it wasn't on the
original mono boards (the added noise was probably entirely due to the
negative inputs having been left floating on that board).

And I'll need to route i2c again, and it's an entirely new untested
configuration.  I've added a trace to route one of the TAC5112 GPIOs
just in case it comes in useful - possibly as an ASI error reporting
interrupt line.

The default codec routing for that new pin being routed is as an
interrupt output: driven low with a weak pull-up.  It's routed to GPIO15
on the rp2354, which hardware in turn defaults to a weak pull-down,
disconnected from any logic.

So without any firmware, this ends up being a few microamps of current
on that trace due to the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
Parts:
- removed C312, C313, C314, C315: 4.7uF, Capacitor_SMD:C_0805_2012Metric, symbol Device:C
- removed U302: TAC5242, Mylib:TAC5242, symbol Mylib:TAC5242
- added J303: AudioJack4, Mylib:PJ-320D, symbol Connector_Audio:AudioJack4
- added R312, R313: 100R, Resistor_SMD:R_0402_1005Metric, symbol Device:R
- added U302: TAC5112, Mylib:TAC5242, symbol Mylib:TAC5212
Connections:
- net +5VA is gone; now on net +3.3VA: C301.2, U301.8 (V+)
- net +3.3VA: now also U302.23 (AVDD); no longer C316.1, C322.1
- net DREG: now also U302.1 (DREG)
- net GND: now also U302.13 (ADDR), U302.A1 (GND), U302.A2 (GND), U302.A3 (GND), U302.A4 (GND), U302.PAD (GND)
- net I2S.BCLK: now also U302.2 (BCLK)
- net I2S.DIN: now also U302.5 (DIN)
- net I2S.DOUT: now also U302.4 (DOUT)
- net I2S.FSYNC: now also U302.3 (FSYNC)
- net IN1M: now also R313.2, U302.16 (IN1M)
- net IN1P: now also C310.2, R309.2, U302.15 (IN1P)
- net IN2M: now also R312.2, U302.18 (IN2M)
- net IN2P: now also C311.2, R310.2, U302.17 (IN2P)
- net MICBIAS: now also R312.1, R313.1, U302.14 (MICBIAS)
- net OUT1P: now also J303.T, U302.20 (OUT1P)
- net OUT2P: now also J303.R1, U302.21 (OUT2P)
- net VREF: now also U302.24 (VREF)
- new net +3V3: C316.1, C322.1, U302.6 (IOVDD)
- new net OUT1M: J303.R2, J303.S, U302.19 (OUT1M), U302.22 (OUT2M)
- new net TAC_GPIO1: U302.9 (GPIO1)
- new net TAC_SCL: U302.7 (SCL)
- new net TAC_SDA: U302.8 (SDA)
Other:
- note added: "Audio connectors and TAC5212 codec"
- note removed: "Audio connector board TAC5242"
- moved on the sheet: C316, C321, C322, C323
